File: hw/bluepill_scsi.sch (KiCad schematic (older format))
At the start: 14 parts, among them J1 Micro_SD_Card, J2 Conn_02x25_Odd_Even, J3 Programming Pins, J4 Berg Power Connector, U1 BluePill_STM32F103C

Commit message: bluescsi-1.0-c-FINAL.zip
Parts:
- D4, D5: footprint Diode_THT:D_A-405_P5.08mm_Vertical_AnodeUp -> Diode_THT:D_A-405_P7.62mm_Horizontal
- J4: symbol 171825-4:171825-4 -> bluepill_scsi-rescue:171825-4-171825-4
Changed lines of the file:
@@
 	2650 5000 1650 5000
 $Comp
-L 171825-4:171825-4 J4
+L bluepill_scsi-rescue:171825-4-171825-4 J4
 U 1 1 5FA7AEFD
 P 2200 5500
@@
 F 0 "D4" V 3096 5770 50  0000 R CNN
 F 1 "Diode" H 3150 5950 50  0000 R CNN
-F 2 "Diode_THT:D_A-405_P5.08mm_Vertical_AnodeUp" H 3050 5850 50  0001 C CNN
+F 2 "Diode_THT:D_A-405_P7.62mm_Horizontal" H 3050 5850 50  0001 C CNN
 F 3 "~" H 3050 5850 50  0001 C CNN
 	1    3050 5850
@@
 F 0 "D5" V 3446 5770 50  0000 R CNN
 F 1 "Diode" H 3450 5950 50  0000 R CNN
-F 2 "Diode_THT:D_A-405_P5.08mm_Vertical_AnodeUp" H 3400 5850 50  0001 C CNN
+F 2 "Diode_THT:D_A-405_P7.62mm_Horizontal" H 3400 5850 50  0001 C CNN
 F 3 "~" H 3400 5850 50  0001 C CNN
 	1    3400 5850
 	0    -1   -1   0
 $EndComp
+$Comp
+L power:VCC #PWR?
+U 1 1 60659E21
+P 8250 1000
+F 0 "#PWR?" H 8250 850 50  0001 C CNN
+F 1 "VCC" H 8265 1173 50  0000 C CNN
+F 2 "" H 8250 1000 50  0001 C CNN
+F 3 "" H 8250 1000 50  0001 C CNN
+	1    8250 1000
+	1    0    0    -1
+$EndComp
 Wire Wire Line
-	8250 1100 8250 850
-Text Label 8250 850  3    50   ~ 0
-TERM_PWR
+	8250 1000 8250 1100
 $EndSCHEMATC

Commit message: Initial 1.1-a
Parts:
- removed J3: Programming Pins, Connector_PinHeader_2.54mm:PinHeader_1x04_P2.54mm_Vertical, symbol Connector_Generic:Conn_01x04
- added H2: MountingHole_Pad, MountingHole:MountingHole_2.7mm_M2.5_Pad_Via, symbol Mechanical:MountingHole_Pad
- added J3: ACT_LED, Connector_PinSocket_2.54mm:PinSocket_1x02_P2.54mm_Vertical, symbol Device:Jumper
- added J4: POWER_LED, Connector_PinSocket_2.54mm:PinSocket_1x02_P2.54mm_Vertical, symbol Device:Jumper
- added R1, R2: R_US, Resistor_THT:R_Axial_DIN0204_L3.6mm_D1.6mm_P5.08mm_Horizontal, symbol Device:R_US
- H1: footprint MountingHole:MountingHole_2.7mm_M2.5 -> MountingHole:MountingHole_2.7mm_M2.5_Pad_Via
- renumbered J4 to J1, J1 to J5
Connections:
- net labels added: EXTERNAL_LED
- wire segments 181 -> 182
