File: hw/bluepill_scsi.kicad_pcb (KiCad board)
At the start: 2 copper layers, 43.8 x 73.7 mm, 14 parts, among them J1 Micro_SD_Card, J2 Conn_02x25_Odd_Even, J3 Programming Pins, J4 Berg Power Connector, U1 BluePill_STM32F103C

Commit message: bluescsi-1.0-c-FINAL.zip
Parts:
- D4, D5: footprint Diode_THT:D_A-405_P5.08mm_Vertical_AnodeUp -> Diode_THT:D_A-405_P7.62mm_Horizontal
- moved D4 2.29 mm to (79.4, 77.9)
- moved D5 2.29 mm to (79.4, 81.4)
Connections:
- H1 pad 1: (no net) -> Net-(H1-Pad1)
- J1 pad 1: (no net) -> Net-(J1-Pad1)
- J1 pad 8: (no net) -> Net-(J1-Pad8)
- J2 pad 25: (no net) -> Net-(J2-Pad25)
- J2 pad 34: (no net) -> Net-(J2-Pad34)
- J4 pad 3: (no net) -> Net-(J4-Pad3)
- J4 pad 4: (no net) -> Net-(J4-Pad4)
- JP2 pad 2: /TERM_PWR -> VCC
- U1 pad 1: (no net) -> Net-(U1-Pad1)
- U1 pad 14: (no net) -> Net-(U1-Pad14)
- U1 pad 17: (no net) -> Net-(U1-Pad17)
- U1 pad 2: (no net) -> /LED
- U1 pad 28: (no net) -> Net-(U1-Pad28)
- U1 pad 29: (no net) -> Net-(U1-Pad29)
- U1 pad 3: (no net) -> Net-(U1-Pad3)
- U1 pad 4: (no net) -> Net-(U1-Pad4)
- U1 pad 5: (no net) -> Net-(U1-Pad5)
- U1 pad 6: (no net) -> Net-(U1-Pad6)
- U1 pad 7: (no net) -> Net-(U1-Pad7)
- U1 pad 8: (no net) -> Net-(U1-Pad8)
Routing:
- net VCC: track 15.5 -> 30.3 mm
- net /TERM_PWR: track 64.6 -> 63.5 mm
- net GND: vias 2 -> 4
Other:
- board text added: "BlueSCSI 1.0-c"
- board text removed: "BlueSCSI 1.0-b"

Commit message: update text
Other:
- board text added: "BlueSCSI(TM) Eric Helgeson - NonCommercial - CC BY-NC 4.0"
Changed lines of the file:
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@@
-(kicad_pcb (version 20171130) (host pcbnew "(5.1.6-0-10_14)")
+(kicad_pcb (version 20171130) (host pcbnew "(5.1.10-1-10_14)")
   (general
     (thickness 1.6)
-    (drawings 12)
+    (drawings 14)
     (tracks 249)
     (zones 0)
@@
     )
   )
+  (gr_text "BlueSCSI(TM) Eric Helgeson - NonCommercial - CC BY-NC 4.0" (at 73.025 110.998 90) (layer B.SilkS)
+    (effects (font (size 1 1) (thickness 0.15)) (justify mirror))
+  )
+  (gr_text "BlueSCSI(TM) Eric Helgeson - NonCommercial - CC BY-NC 4.0" (at 73.025 110.998 90) (layer F.SilkS)
+    (effects (font (size 1 1) (thickness 0.15)))
+  )
   (gr_line (start 71.755 149.225) (end 71.12 149.225) (layer Edge.Cuts) (width 0.05))
