File: hw/desktop-50-pin/bluepill_scsi.kicad_pcb (KiCad board)
At the start: 2 copper layers, 43.8 x 73.7 mm, 23 parts, among them J1 Berg Power Connector, J2 Conn_02x25_Odd_Even, J3 ACT_LED, J4 POWER_LED, J5 Micro_SD_Card, U1 BluePill_STM32F103C

Commit message: 1.1-a
Parts:
- removed the G*** at (82.8, 112.9)
Routing:
- net GND: vias 1 -> 4
Other:
- board text added: "BlueSCSI(TM) © Eric Helgeson 2021 github.com/erichelgeson/bluescsi"
- board text removed: "500-1kΩ"
- board text removed: "BlueSCSI(TM) © Eric Helgeson github.com/erichelgeson/bluescsi"
