File: hw/external-db25/bluepill_scsi.kicad_pcb (KiCad board)
At the start: 2 copper layers, 37.3 x 54.1 mm, 11 parts, among them J2 DB25_Male_MountingHoles, J5 Micro_SD_Card, U1 BluePill_STM32F103C

Commit message: 1.1-a
Connections:
- J2 pad 0: Net-(J2-Pad0) -> GND
Routing:
- net +3V3: track 64.3 -> 12.4 mm, vias 2 -> 1
- net /SCSI_DAT3: track 34.0 -> 20.7 mm, vias 0 -> 1
- net /SCSI_DAT4: track 49.9 -> 41.9 mm, vias 2 -> 0
- net /TERM_PWR: track 65.0 -> 69.2 mm
- net /SCSI_DAT5: track 36.1 -> 37.5 mm
- net /SCSI_DBP: track 45.3 -> 46.5 mm
- net GND: vias 0 -> 4
- net /SCSI_DAT6: vias 0 -> 1
- net (no net): vias 1 -> 0
