File: hw/external-db25/bluepill_scsi.sch (KiCad schematic (older format))
At the start: 8 parts, among them J2 DB25_Male_MountingHoles, J5 Micro_SD_Card, U1 BluePill_STM32F103C

Commit message: 1.1-a
Connections:
- wire segments 126 -> 130
Changed lines of the file:
@@
 $EndComp
 Wire Wire Line
-	6200 1400 6200 1200
+	6200 1400 6200 1250
 Wire Wire Line
 	5500 1400 6200 1400
@@
 Wire Wire Line
 	7900 1000 7900 1800
+Wire Wire Line
+	5200 1100 6050 1100
+Wire Wire Line
+	6050 1100 6050 1250
+Wire Wire Line
+	6050 1250 6200 1250
+Connection ~ 6200 1250
+Wire Wire Line
+	6200 1250 6200 1200
 $EndSCHEMATC
