File: cc-nc-hardware/PowerBook/LED_Indicators.kicad_sch (KiCad schematic)
At the start: 7 parts, among them U8 74HC14

Commit message: PowerBook Hardware Version 2023.10a
Connections:
- net oBSY: now also U8.3
- net at R30.1, U8.2: no longer U8.3
Other:
- note added: "BlueSCSI V2, PowerBook 2023_10a"
- note added: "External Activity LED"
- note added: "October 2023"
- note added: "Unused Inverter Pins"
- note added: "© 2022 - 2023 Tech by Androda, LLC Licensed Attribution-NonCommercial-ShareAlike 4.0 International (CC BY-NC-SA 4.0) https://creativecommons.org/licenses/by-nc-sa/4.0/legalcode"
- moved on the sheet: U8C, U8D, U8E, U8F, U8G
