File: cc-nc-hardware/PowerBook/PowerBook.kicad_sch (KiCad schematic)
At the start: 91 parts, among them J1 Conn_01x03_Male, J2 PB_SCSI_HD_Pins, J4 SW, J6 Conn_01x02_Male, SW1 SW_MEC_5E, U1 SN74CBTD3384, U2 SN74CBTD3384, U3 AMS1117-2.85, U4 LVT245, U5 LVT125, U6 LVT125, U7 LVT125, U9 LVT245

Commit message: PowerBook Hardware Version 2023.10a
Parts:
- removed H4: MountingHole, MountingHole:MountingHole_3.2mm_M3, symbol Mechanical:MountingHole
- removed J4: SW, Connector_PinHeader_2.54mm:PinHeader_2x02_P2.54mm_Vertical, symbol Connector_Generic:Conn_02x02_Odd_Even
- removed J6: Conn_01x02_Male, Connector_PinHeader_2.54mm:PinHeader_1x02_P2.54mm_Vertical, symbol Connector:Conn_01x02_Male
- removed R24, R26, R27: 1k, Resistor_SMD:R_0603_1608Metric_Pad0.98x0.95mm_HandSolder, symbol Device:R
- removed R31, R32: 4.7k, Resistor_SMD:R_0603_1608Metric_Pad0.98x0.95mm_HandSolder, symbol Device:R
- removed R43, R44, R45, R46, R47, R48, R49, R50, R51, R52, R53, R54, R55: 1k, Resistor_SMD:R_0402_1005Metric_Pad0.72x0.64mm_HandSolder, symbol Device:R
- removed SW1: SW_MEC_5E, Library:TS-1187A-B-A-B, symbol Switch:SW_MEC_5E
- removed U1, U2: SN74CBTD3384, Package_SO:TSSOP-24_4.4x7.8mm_P0.65mm, symbol New_Library:SN74CBTD3384
- added C1: 0.1uF, Capacitor_SMD:C_0805_2012Metric_Pad1.18x1.45mm_HandSolder, symbol Device:C
- added C16: 0.1uF, Capacitor_SMD:C_0805_2012Metric, symbol Device:CP
- added J3: SM04B-SRSS-TB(LF)(SN), Library:JST_SM04B-SRSS-TB(LF)(SN), symbol New_Library:SM04B-SRSS-TB(LF)(SN)
- added Q1, Q2: AO3401A, Package_TO_SOT_SMD:SOT-23, symbol Transistor_FET:AO3401A
- added U1, U2: LVT245, Package_SO:TSSOP-20_4.4x6.5mm_P0.65mm, symbol New_Library:LVT245
- C12, C7: footprint Capacitor_SMD:C_0805_2012Metric_Pad1.18x1.45mm_HandSolder -> Capacitor_SMD:C_0805_2012Metric
- R1, R10, R2, R3, R33, R34, R35, R36, R37, R38, R39, R4, R40, R5, R6, R7, R8, R9: value R -> 110
- R11: value 1k -> 4.7k; footprint Resistor_SMD:R_0402_1005Metric_Pad0.72x0.64mm_HandSolder -> Resistor_SMD:R_0603_1608Metric
- R20: value 10k -> 4.7k; footprint Resistor_SMD:R_0603_1608Metric_Pad0.98x0.95mm_HandSolder -> Resistor_SMD:R_0603_1608Metric
- R21: value 10k -> 1k; footprint Resistor_SMD:R_0603_1608Metric_Pad0.98x0.95mm_HandSolder -> Resistor_SMD:R_0603_1608Metric
- R22: value 10k -> 1k
- RP1: footprint CustomFootprints:BluePillModule -> Library:Raspberry_Pi_PicoW_SMT_THT
- U4, U9: value LVT245 -> LVTH245
Connections:
- net oRST is gone; now on net GND: U5.1 (1/OE), U5.2 (1A)
- net +2V8: now also R23.2, Q1.2 (S), Q2.2 (S), U1.1 (DIR), U1.2 (A1), U1.20 (Vcc), U1.3 (A2), U1.4 (A3), U1.5 (A4), U1.6 (A5), U1.7 (A6), U1.8 (A7), U1.9 (A8), U2.1 (DIR), U2.2 (A1), U2.20 (Vcc), U2.3 (A2), U2.4 (A3), U2.5 (A4), U2.6 (A5), U2.7 (A6), U2.8 (A7), U2.9 (A8); no longer R20.2, R21.2
- net +3V3: now also R11.2, R20.1, C1.2, C16.1, J3.2
- net GND: now also C1.1, C16.2, J3.1, J3.S1 (SHIELD), J3.S2 (SHIELD), U1.10 (GND), U2.10 (GND); no longer R11.1, R23.2
- net RST: no longer U5.3 (1Y)
- net TRM_ON_J: now also Q1.1 (G), Q2.1 (G), U1.19 (/OE), U2.19 (/OE)
- net iRST: now also R21.1; no longer RP1.27 (G21)
- net oIO: no longer R20.1
- net oREQ: now also RP1.25 (G19); no longer R21.1, RP1.22 (G17)
- net oSEL: now also R21.2, RP1.27 (G21); no longer RP1.25 (G19)
- net at R39.1: now also U1.13 (B6)
- net at R34.1: now also U1.17 (B2)
- net at R10.1: now also U2.15 (B4)
- net at R7.1: now also U2.18 (B1)
- net at R37.1: now also U1.11 (B8)
- net at R2.1: now also U2.11 (B8)
- net at R9.1: now also U2.16 (B3)
- net at R8.1: now also U2.17 (B2)
- net at R6.1: now also Q1.3 (D)
- net at R5.1: now also U2.14 (B5)
- net at R4.1: now also U2.13 (B6)
- net at R3.1: now also U2.12 (B7)
- net at R40.1: now also U1.14 (B5)
- net at R1.1: now also U1.15 (B4)
- net at R38.1: now also U1.12 (B7)
- net at R35.1: now also U1.18 (B1)
- net at R36.1: now also Q2.3 (D)
- net at R33.1: now also U1.16 (B3)
- net at U4.3 (A2): no longer R11.2
- net SERIAL_OUT renamed SDA
- net SDA: now also R11.1, J3.3
- new net SCL: J3.4, R20.2, RP1.22 (G17)
Other:
- note added: "Active SCSI Termination"
- note added: "BlueSCSI V2, PowerBook 2023_10a"
- note added: "Data Bus Transceivers"
- note added: "Decoupling Capacitors"
- note added: "External I2C "qwiic" by SparkFun"
- note added: "MicroSD Card"
- note added: "October 2023"
- note added: "PUP Necessary"
- note added: "Power Distribution"
- note added: "Raspberry Pi Pico (or W)"
- note added: "SCSI Connector"
- note added: "SCSI Control Line Bus Buffers"
- note added: "SM04B-SRSS-TB(LF)(SN) Symbol And Footprint Copyright SnapEDA https://www.snapeda.com/parts/SM04B-SRSS-TB%28LF%29%28SN%29/JST%20Sales/view-part/ License For This Symbol and Footprint Only: CC-BY-SA 4.0 https://creativecommons.org/licenses/by-sa/4.0/ This license contains a warranty disclaimer, please read it in full"
- note added: "Termination Power"
- note added: "© 2022 - 2023 Tech by Androda, LLC Licensed Attribution-NonCommercial-ShareAlike 4.0 International (CC BY-NC-SA 4.0) https://creativecommons.org/licenses/by-nc-sa/4.0/legalcode"
- note removed: "1k Drain Resistors Necessary LVT, Omit LVTH"
- note removed: "BlueSCSI V2, PowerBook V1"
- note removed: "November 2022"
- note removed: "Opt. PUP Didn't need them"
- note removed: "RUN is the RP2040 enable pin, and has an internal (on-chip) pull-up resistor to 3.3V of about ~50kΩ. To reset RP2040, short this pin low."
- note removed: "© 2022 Tech by Androda, LLC Licensed Attribution-NonCommercial-ShareAlike 4.0 International (CC BY-NC-SA 4.0) https://creativecommons.org/licenses/by-nc-sa/4.0/legalcode"
- moved on the sheet: C10, C11, C12, C13, C14, C15, C2, C3, C4, C5, C6, C7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
