File: cc-nc-hardware/Desktop_50_Pin/Desktop_50_Pin_TopConn.kicad_pcb (KiCad board)
At the start: 2 copper layers, 93.7 x 82.6 mm, 101 parts, among them J1 Conn_01x03_Male, J2 Conn_02x25_Odd_Even, J3 BergFloppy, J4 SW, J5 Conn_01x03_Male, J6 Conn_01x02_Male, J7 TERM_BCKF, J8 EPWR, J9 Conn_01x02_Male, SW1 SW_MEC_5E, U1 SN74CBTD3384, U2 SN74CBTD3384, U3 AMS1117-2.85, U4 LVT245, U5 LVT125, U6 LVT125, U7 LVT125, U8 74HC14, U9 LVT245

Commit message: Desktop PCB Version 2023.03a
Parts:
- removed R57: 470, Resistor_SMD:R_0402_1005Metric_Pad0.72x0.64mm_HandSolder
- added JP1: SolderJumper_2_Open, Jumper:SolderJumper-2_P1.3mm_Open_RoundedPad1.0x1.5mm, F.Cu at (181.4, 80.3)
- added JP2: SolderJumper_2_Open, Jumper:SolderJumper-2_P1.3mm_Open_RoundedPad1.0x1.5mm, F.Cu at (185.3, 80.3)
- added R58: 150, Resistor_SMD:R_0603_1608Metric_Pad0.98x0.95mm_HandSolder, F.Cu at (181.4, 78.1)
- added R59: 330, Resistor_SMD:R_0603_1608Metric_Pad0.98x0.95mm_HandSolder, F.Cu at (185.3, 78.1)
- moved C7 36.3 mm to (188.4, 119.6)
- moved C6 13.2 mm to (188.5, 68.1)
- moved J7 2.35 mm to (184.6, 72.4), turned to 180 degrees
- moved G*** 0.38 mm to (122.4, 143.3)
Routing:
- net GND: track 1407.1 -> 1451.6 mm, vias 112 -> 114
- net Net-(JP1-Pad2): track 0.00 -> 10.5 mm
- net Net-(F3-Pad2): track 8.57 -> 3.43 mm
- net +5V: track 130.0 -> 134.4 mm
- net Net-(C7-Pad1): track 81.4 -> 80.2 mm
- net +5VP: track 117.8 -> 116.9 mm
- net Net-(JP1-Pad1): track 38.5 -> 39.4 mm
- net Net-(J5-Pad2): track 6.46 -> 7.19 mm
Other:
- board text added: "V2 - 2023.03a"
- board text removed: "V2 - 2022.12a"

Commit message: Desktop 2023.09a Hardware Design
Parts:
- removed R27: 1k, Resistor_SMD:R_0603_1608Metric_Pad0.98x0.95mm_HandSolder
- removed R31, R32: 4.7k, Resistor_SMD:R_0603_1608Metric_Pad0.98x0.95mm_HandSolder
- removed R43, R44, R45, R46, R47, R48, R49, R50, R51, R52, R53, R54, R55: 1k, Resistor_SMD:R_0402_1005Metric_Pad0.72x0.64mm_HandSolder
- removed U1, U2: SN74CBTD3384, Package_SO:TSSOP-24_4.4x7.8mm_P0.65mm
- removed U7: LVT125, Package_SO:TSSOP-14_4.4x5mm_P0.65mm
- added C17: 0.1uF, Capacitor_SMD:C_0805_2012Metric, F.Cu at (116.7, 112.7)
- added C18: 0.1uF, Capacitor_SMD:C_0805_2012Metric, F.Cu at (113.4, 79.2)
- added C19: 0.1uF, Capacitor_SMD:C_0805_2012Metric_Pad1.18x1.45mm_HandSolder, F.Cu at (136.6, 72.5)
- added C20: 0.1uF, Capacitor_SMD:C_0805_2012Metric_Pad1.18x1.45mm_HandSolder, F.Cu at (143.1, 107.2)
- added C21: 4.7uF, Capacitor_SMD:C_0805_2012Metric_Pad1.18x1.45mm_HandSolder, F.Cu at (131.6, 106.3)
- added C22: 0.1uF, Capacitor_SMD:C_0805_2012Metric_Pad1.18x1.45mm_HandSolder, F.Cu at (185.2, 71.0)
- added C23: 4.7uF, Capacitor_SMD:C_0805_2012Metric_Pad1.18x1.45mm_HandSolder, F.Cu at (178.0, 124.0)
- added D5: D, Diode_SMD:D_SMA, F.Cu at (182.1, 141.8)
- added G***: LOGO, LOGO, F.Cu at (190.0, 73.6)
- added J10: Conn_01x03_Male, Connector_PinHeader_2.54mm:PinHeader_1x03_P2.54mm_Vertical, F.Cu at (140.5, 79.1)
- added J11: Conn_01x02_Male, Connector_PinHeader_2.54mm:PinHeader_1x02_P2.54mm_Vertical, F.Cu at (128.7, 107.5)
- added Q1: AO3401A, Package_TO_SOT_SMD:SOT-23, F.Cu at (118.5, 79.4)
- added Q2: AO3401A, Package_TO_SOT_SMD:SOT-23, F.Cu at (117.3, 118.9)
- added R20: 5.1k, Resistor_SMD:R_0402_1005Metric, F.Cu at (184.7, 140.3)
- added R21: 5.1k, Resistor_SMD:R_0402_1005Metric, F.Cu at (184.3, 135.0)
- added R22: 4.7k, Resistor_SMD:R_0603_1608Metric, F.Cu at (136.2, 93.8)
- added R61: 1k, Resistor_SMD:R_0402_1005Metric, F.Cu at (147.6, 108.2)
- added R65: 1k, Resistor_SMD:R_0402_1005Metric, F.Cu at (146.6, 80.4)
- added R66: 1k, Resistor_SMD:R_0402_1005Metric, F.Cu at (138.4, 92.7)
- added R67: 1k, Resistor_SMD:R_0402_1005Metric, F.Cu at (146.9, 96.9)
- added R68: 1k, Resistor_SMD:R_0402_1005Metric, F.Cu at (147.7, 89.8)
- added R69: 1k, Resistor_SMD:R_0402_1005Metric, F.Cu at (147.6, 109.3)
- added SD2: MicroSD-TF-06, Library:TF-06_MicroSD, F.Cu at (191.5, 123.5)
- added U13: LVT125, Package_SO:TSSOP-14_4.4x5mm_P0.65mm, F.Cu at (130.4, 73.9)
- added U14: LVT125, Package_SO:TSSOP-14_4.4x5mm_P0.65mm, F.Cu at (130.5, 81.8)
- added U15: LVT125, Package_SO:TSSOP-14_4.4x5mm_P0.65mm, F.Cu at (130.5, 89.7)
- added U16: LVT125, Package_SO:TSSOP-14_4.4x5mm_P0.65mm, F.Cu at (130.5, 97.7)
- J4: value SW -> USB_C_Receptacle; footprint Connector_PinHeader_2.54mm:PinHeader_2x02_P2.54mm_Vertical -> Connector_USB:USB_C_Receptacle_HRO_TYPE-C-31-M-12
- J6: value Conn_01x02_Male -> SM04B-SRSS-TB(LF)(SN); footprint Connector_PinHeader_2.54mm:PinHeader_1x02_P2.54mm_Vertical -> Library:JST_SM04B-SRSS-TB(LF)(SN)
- R1, R10, R2, R3, R33, R34, R35, R36, R37, R38, R39, R4, R40, R5, R6, R7, R8, R9: value R -> 110
- R11: footprint Resistor_SMD:R_0402_1005Metric_Pad0.72x0.64mm_HandSolder -> Resistor_SMD:R_0402_1005Metric
- R23, R24, R26: value 1k -> 4.7k; footprint Resistor_SMD:R_0603_1608Metric_Pad0.98x0.95mm_HandSolder -> Resistor_SMD:R_0603_1608Metric
- R25, R28, R29: footprint Resistor_SMD:R_0603_1608Metric_Pad0.98x0.95mm_HandSolder -> Resistor_SMD:R_0402_1005Metric
- RP1: value Pico_Footprint -> PicoWModule; footprint CustomFootprints:BluePillModule -> Library:Raspberry_Pi_PicoW_SMT_THT
- U5, U6: value LVT125 -> LVT245; footprint Package_SO:TSSOP-14_4.4x5mm_P0.65mm -> Package_SO:TSSOP-20_4.4x6.5mm_P0.65mm
- moved R24 63.6 mm to (184.4, 68.4)
- moved R26 56.6 mm to (184.4, 66.6), turned to 0 degrees
- moved J4 54.6 mm to (190.8, 137.4), turned to 90 degrees
- moved U6 53.5 mm to (117.3, 124.4)
- moved D4 53.2 mm to (140.3, 110.6)
- moved D3 53.0 mm to (140.1, 113.8)
- moved R56 52.7 mm to (136.8, 110.6)
- moved R30 51.9 mm to (137.0, 113.6)
- moved F2 50.9 mm to (129.3, 67.4), turned to 180 degrees
- moved R11 49.6 mm to (138.9, 84.5), turned to 0 degrees
- moved G*** 39.6 mm to (161.6, 138.0)
- moved R41 36.8 mm to (115.6, 79.4), turned to -90 degrees
- moved U8 34.0 mm to (137.4, 105.7), turned to -90 degrees
- moved R14 30.5 mm to (138.3, 120.4), turned to 180 degrees
- moved R12 30.5 mm to (138.3, 118.2), turned to 180 degrees
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Connections:
- J6 pad 1: SERIAL_OUT -> GND
- J6 pad 2: GND -> +3V3
- R11 pad 1: GND -> iSEL
- R11 pad 2: Net-(R11-Pad2) -> Net-(J10-Pad3)
- R23 pad 2: GND -> +2V8
- R24 pad 1: oRST -> SDA
- R24 pad 2: +2V8 -> +3V3
- R26 pad 1: Net-(J4-Pad1) -> +3V3
- R26 pad 2: GND -> SCL
- R28 pad 1: oCD_iSEL -> iCD
- R28 pad 2: SEL_BUFF -> Net-(J10-Pad1)
- R29 pad 1: BSY_BUFF -> iBSY
- RP1 pad 21: SERIAL_OUT -> SDA
- RP1 pad 22: oREQ -> SCL
- RP1 pad 25: oSEL -> oREQ
- RP1 pad 27: iRST -> oSEL
- RP1 pad 31: iACK -> oACK
- RP1 pad 34: iATN -> Net-(R61-Pad1)
- SW1 pad 1: oRST -> GND
- SW1 pad 2: GND -> RST
- U4 pad 12: Net-(R49-Pad1) -> unconnected-(U4-Pad12)
- U4 pad 14: Net-(R48-Pad1) -> unconnected-(U4-Pad14)
- U4 pad 15: Net-(R47-Pad1) -> unconnected-(U4-Pad15)
- U4 pad 17: Net-(R46-Pad1) -> unconnected-(U4-Pad17)
- U4 pad 3: Net-(R11-Pad2) -> unconnected-(U4-Pad3)
- U4 pad 5: Net-(R43-Pad2) -> unconnected-(U4-Pad5)
- U4 pad 6: Net-(R44-Pad2) -> unconnected-(U4-Pad6)
- U4 pad 8: Net-(R45-Pad2) -> unconnected-(U4-Pad8)
- U5 pad 1: oRST -> +2V8
- U5 pad 10: oBSY -> GND
- U5 pad 11: BSY -> Net-(R2-Pad1)
- U5 pad 12: oBSY -> Net-(R3-Pad1)
- U5 pad 13: oBSY -> Net-(R4-Pad1)
- U5 pad 14: +2V8 -> Net-(R5-Pad1)
- U5 pad 2: oRST -> +2V8
- U5 pad 3: RST -> +2V8
- U5 pad 4: oBSY -> +2V8
- U5 pad 5: ACK -> +2V8
- U5 pad 6: iACK -> +2V8
- U5 pad 7: GND -> +2V8
- U5 pad 8: iATN -> +2V8
- U5 pad 9: ATN -> +2V8
- U6 pad 1: GND -> +2V8
- U6 pad 10: oREQ -> GND
- U6 pad 11: IO -> Net-(R36-Pad1)
- U6 pad 12: oIO -> Net-(R37-Pad1)
- U6 pad 13: oIO -> Net-(R38-Pad1)
- U6 pad 14: +2V8 -> Net-(R39-Pad1)
- U6 pad 2: SEL -> +2V8
- U6 pad 3: SEL_BUFF -> +2V8
- U6 pad 4: GND -> +2V8
- U6 pad 5: BSY -> +2V8
- U6 pad 6: BSY_BUFF -> +2V8
- U6 pad 7: GND -> +2V8
- U6 pad 8: REQ -> +2V8
- U6 pad 9: oREQ -> +2V8
- U8 pad 3: GND -> oBSY
- U8 pad 4: unconnected-(U8-Pad4) -> !oBSY
- U9 pad 12: Net-(R55-Pad1) -> unconnected-(U9-Pad12)
- U9 pad 15: Net-(R54-Pad1) -> unconnected-(U9-Pad15)
- U9 pad 17: Net-(R53-Pad1) -> unconnected-(U9-Pad17)
- U9 pad 3: Net-(R50-Pad2) -> unconnected-(U9-Pad3)
- U9 pad 5: Net-(R51-Pad2) -> unconnected-(U9-Pad5)
- U9 pad 8: Net-(R52-Pad2) -> unconnected-(U9-Pad8)
Routing:
- net GND: track 1451.6 -> 569.8 mm, vias 114 -> 100
- net +3V3: track 52.4 -> 149.2 mm, vias 0 -> 4
- net SCL: track 0.00 -> 50.3 mm, vias 0 -> 1
- net +5F: track 169.3 -> 121.4 mm, vias 0 -> 3
- net !oBSY: track 0.00 -> 47.5 mm, vias 0 -> 10
- net SDA: track 0.00 -> 44.8 mm, vias 0 -> 1
- net +2V8: track 311.1 -> 270.2 mm, vias 6 -> 11
- net Net-(R17-Pad1): track 5.24 -> 43.4 mm
- net +5VP: track 116.9 -> 154.4 mm
- net Net-(R14-Pad1): track 4.45 -> 40.2 mm
- net USB_DM: track 0.00 -> 35.5 mm, vias 0 -> 2
- net SD_D3_CS: track 23.2 -> 58.1 mm, vias 0 -> 2
- net Net-(R15-Pad1): track 4.94 -> 39.2 mm
- net Net-(R12-Pad1): track 5.89 -> 40.0 mm
- net SD_D2: track 16.6 -> 50.7 mm, vias 0 -> 2
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- added copper zone on In1.Cu, net GND
- added copper zone on In2.Cu, net GND
Other:
- outline, holes or cut-outs redrawn
- copper layers 2 -> 4
- board text added: "BlueSCSI © Eric Helgeson PCB © Tech by Androda, LLC CC BY-NC-SA 4.0 NOT FOR COMMERCIAL SALE"
- board text added: "Initiator"
- board text added: "JLCJLCJLCJLC"
- board text added: "Target"
- board text added: "Use Only One SD Slot"
- board text added: "V2 - 2023.09a"
- board text removed: "BlueSCSI © Eric Helgeson"
- board text removed: "CC BY-NC-SA 4.0 NOT FOR COMMERCIAL SALE"
- board text removed: "PCB © Tech by Androda, LLC"
- board text removed: "S1"
- board text removed: "S2"
- board text removed: "SDBG"
- board text removed: "V2 - 2023.03a"
- board text removed: "https://bluescsi.com"

Commit message: Desktop 2023.10a design
Parts:
- removed D5: D, Diode_SMD:D_SMA
- removed J4: USB_C_Receptacle, Connector_USB:USB_C_Receptacle_HRO_TYPE-C-31-M-12
- removed R20, R21: 5.1k, Resistor_SMD:R_0402_1005Metric
- removed SD2: MicroSD-TF-06, Library:TF-06_MicroSD
- added C24: 0.1uF, Capacitor_SMD:C_0805_2012Metric_Pad1.18x1.45mm_HandSolder, F.Cu at (172.1, 118.3)
- C23: value 4.7uF -> 20uF; footprint Capacitor_SMD:C_0805_2012Metric_Pad1.18x1.45mm_HandSolder -> Capacitor_SMD:C_1206_3216Metric
- J11: value Conn_01x02_Male -> ACK_En
- moved C16 67.7 mm to (159.3, 68.5)
- moved D2 67.7 mm to (154.0, 73.3)
- moved J8 67.7 mm to (153.1, 68.6)
- moved J9 67.7 mm to (153.1, 78.6)
- moved C7 57.7 mm to (160.7, 76.8)
- moved R61 20.4 mm to (135.6, 91.6)
- moved R69 20.4 mm to (135.6, 92.7)
- moved R68 18.4 mm to (135.1, 76.4), turned to 90 degrees
- moved R67 17.1 mm to (133.4, 107.3)
- moved RP1 16.2 mm to (156.1, 119.8)
- moved R29 16.1 mm to (138.2, 105.8)
- moved H3 15.1 mm to (136.1, 142.6)
- moved C23 14.9 mm to (169.7, 136.4)
- moved G*** 14.0 mm to (170.6, 127.2), turned to 90 degrees
- moved R65 12.8 mm to (135.9, 73.3), turned to 90 degrees
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Connections:
- C23 pad 1: +3V3 -> +5VP
Routing:
- net GND: track 569.8 -> 946.8 mm, vias 100 -> 81
- net Net-(D2-Pad2): track 70.1 -> 151.4 mm, vias 0 -> 3
- net SD_D3_CS: track 58.1 -> 4.21 mm, vias 2 -> 0
- net SD_D1: track 59.6 -> 10.7 mm, vias 3 -> 0
- net +3V3: track 149.2 -> 109.8 mm, vias 4 -> 6
- net SD_D2: track 50.7 -> 11.5 mm, vias 2 -> 0
- net Net-(R61-Pad1): track 7.97 -> 46.5 mm
- net SD_D0_MISO: track 54.6 -> 16.3 mm, vias 3 -> 0
- net Net-(C7-Pad1): track 82.0 -> 45.2 mm, vias 3 -> 0
- net USB_DM: track 35.5 -> 0.00 mm, vias 2 -> 0
- net USB_DP: track 33.0 -> 0.00 mm, vias 2 -> 0
- net oMSG_iBSY: track 25.4 -> 58.0 mm
- net SD_CLK: track 45.1 -> 13.1 mm, vias 2 -> 1
- net SD_CMD_MOSI: track 44.9 -> 16.0 mm, vias 2 -> 1
- net +5F: track 121.4 -> 93.3 mm, vias 3 -> 6
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- removed copper zone on In1.Cu, net GND
- removed copper zone on In2.Cu, net GND
Other:
- board size 93.7 x 82.6 mm -> 89.2 x 82.6 mm
- copper layers 4 -> 2
- board text added: "V2 - 2023.10a"
- board text added: "© 2022 - 2023 Tech by Androda, LLC Licensed Attribution-NonCommercial-ShareAlike 4.0 International (CC BY-NC-SA 4.0) https://creativecommons.org/licenses/by-nc-sa/4.0/legalcode"
- board text removed: "Use Only One SD Slot"
- board text removed: "V2 - 2023.09a"
