File: cc-nc-hardware/Desktop_50_Pin/Desktop_50_Pin_TopConn.kicad_sch (KiCad schematic)
At the start: 96 parts, among them J1 Conn_01x03_Male, J2 Conn_02x25_Odd_Even, J3 BergFloppy, J4 SW, J6 Conn_01x02_Male, J7 TERM_BCKF, J8 EPWR, J9 Conn_01x02_Male, SW1 SW_MEC_5E, U1 SN74CBTD3384, U2 SN74CBTD3384, U3 AMS1117-2.85, U4 LVT245, U5 LVT125, U6 LVT125, U7 LVT125, U9 LVT245

Commit message: Desktop PCB Version 2023.03a
Other:
- note added: "BlueSCSI V2, Desktop 50 Pin, Top Connector, 2023.03a"
- note added: "March 2023"
- note added: "© 2023 Tech by Androda, LLC Licensed Attribution-NonCommercial-ShareAlike 4.0 International (CC BY-NC-SA 4.0) https://creativecommons.org/licenses/by-nc-sa/4.0/legalcode"
- note removed: "BlueSCSI V2, Desktop 50 Pin, Top Connector, 2022_12a"
- note removed: "December 2022"
- note removed: "© 2022 Tech by Androda, LLC Licensed Attribution-NonCommercial-ShareAlike 4.0 International (CC BY-NC-SA 4.0) https://creativecommons.org/licenses/by-nc-sa/4.0/legalcode"
Changed lines of the file:
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@@
     (effects (font (size 1.27 1.27)) (justify left bottom))
   )
-  (text "December 2022" (at 205.74 194.31 0)
+  (text "March 2023" (at 205.74 194.31 0)
     (effects (font (size 1.27 1.27)) (justify left bottom))
   )
-  (text "© 2022 Tech by Androda, LLC\nLicensed Attribution-NonCommercial-ShareAlike 4.0 International (CC BY-NC-SA 4.0)\nhttps://creativecommons.org/licenses/by-nc-sa/4.0/legalcode"
-    (at 177.8 173.99 0)
-    (effects (font (size 1.27 1.27)) (justify left bottom))
-  )
-  (text "BlueSCSI V2, Desktop 50 Pin, Top Connector, 2022_12a"
+  (text "BlueSCSI V2, Desktop 50 Pin, Top Connector, 2023.03a"
     (at 186.69 190.5 0)
     (effects (font (size 1.27 1.27)) (justify left bottom))
@@
     (effects (font (size 1.27 1.27)) (justify left bottom))
   )
+  (text "© 2023 Tech by Androda, LLC\nLicensed Attribution-NonCommercial-ShareAlike 4.0 International (CC BY-NC-SA 4.0)\nhttps://creativecommons.org/licenses/by-nc-sa/4.0/legalcode"
+    (at 177.8 173.99 0)
+    (effects (font (size 1.27 1.27)) (justify left bottom))
+  )
   (text "PDN Necessary" (at 115.57 171.45 0)
     (effects (font (size 1.27 1.27)) (justify left bottom))
@@
       (reference "J9") (unit 1) (value "Conn_01x02_Male") (footprint "Connector_PinHeader_2.54mm:PinHeader_1x02_P2.54mm_Vertical")
     )
+    (path "/d5fc13d4-1ca0-477a-91ea-84605f39f5f9/2de70ce8-1ae0-4c74-b56f-c1191fa8e250"
+      (reference "JP1") (unit 1) (value "SolderJumper_2_Open") (footprint "Jumper:SolderJumper-2_P1.3mm_Open_RoundedPad1.0x1.5mm")
+    )
+    (path "/d5fc13d4-1ca0-477a-91ea-84605f39f5f9/2e4317c4-aac7-453f-a079-7fbec4fe7cb0"
+      (reference "JP2") (unit 1) (value "SolderJumper_2_Open") (footprint "Jumper:SolderJumper-2_P1.3mm_Open_RoundedPad1.0x1.5mm")
+    )
     (path "/d55cc04d-788a-42ba-a149-99196a85fed4"
       (reference "R1") (unit 1) (value "R") (footprint "Resistor_SMD:R_0603_1608Metric_Pad0.98x0.95mm_HandSolder")
@@
       (reference "R57") (unit 1) (value "470") (footprint "Resistor_SMD:R_0402_1005Metric_Pad0.72x0.64mm_HandSolder")
     )
+    (path "/d5fc13d4-1ca0-477a-91ea-84605f39f5f9/0e7581f4-5fdd-4863-a8e3-8d5161063b63"
+      (reference "R58") (unit 1) (value "150") (footprint "Resistor_SMD:R_0603_1608Metric_Pad0.98x0.95mm_HandSolder")
+    )
+    (path "/d5fc13d4-1ca0-477a-91ea-84605f39f5f9/03142d3f-f27d-4d9f-9f6c-b0498a9f3df9"
+      (reference "R59") (unit 1) (value "330") (footprint "Resistor_SMD:R_0603_1608Metric_Pad0.98x0.95mm_HandSolder")
+    )
     (path "/00000000-0000-0000-0000-000060ad3c40"

Commit message: Desktop 2023.09a Hardware Design
Parts:
- removed C1, C2, C5: 0.1uF, Capacitor_SMD:C_0805_2012Metric_Pad1.15x1.40mm_HandSolder, symbol Device:CP
- removed C10, C15: 4.7uF, Capacitor_SMD:C_0805_2012Metric_Pad1.18x1.45mm_HandSolder, symbol Device:CP
- removed C11, C13, C14, C8, C9: 0.1uF, Capacitor_SMD:C_0805_2012Metric_Pad1.18x1.45mm_HandSolder, symbol Device:C
- removed C12, C6: 4.7uF, Capacitor_SMD:C_0805_2012Metric_Pad1.15x1.40mm_HandSolder, symbol Device:CP
- removed C16: 4.7uF, Capacitor_SMD:C_0805_2012Metric_Pad1.18x1.45mm_HandSolder, symbol Device:C
- removed C3, C4: 20uF, Capacitor_SMD:C_1206_3216Metric_Pad1.42x1.75mm_HandSolder, symbol Device:CP
- removed C7: 4.7uF, Capacitor_SMD:C_0805_2012Metric_Pad1.15x1.40mm_HandSolder, symbol Device:C
- removed D1, D2: D, Diode_SMD:D_SMA, symbol Device:D
- removed F2, F3: Polyfuse, Fuse:Fuse_0805_2012Metric_Pad1.15x1.40mm_HandSolder, symbol Device:Polyfuse
- removed J1: Conn_01x03_Male, Connector_PinHeader_2.54mm:PinHeader_1x03_P2.54mm_Vertical, symbol Connector:Conn_01x03_Male
- removed J2: Conn_02x25_Odd_Even, Connector_PinHeader_2.54mm:PinHeader_2x25_P2.54mm_Horizontal, symbol Connector_Generic:Conn_02x25_Odd_Even
- removed J3: BergFloppy, CustomFootprints:BergFloppy_RightAngle, symbol custom_symbols:BergFloppy
- removed J4: SW, Connector_PinHeader_2.54mm:PinHeader_2x02_P2.54mm_Vertical, symbol Connector_Generic:Conn_02x02_Odd_Even
- removed J6, J9: Conn_01x02_Male, Connector_PinHeader_2.54mm:PinHeader_1x02_P2.54mm_Vertical, symbol Connector:Conn_01x02_Male
- removed J7: TERM_BCKF, Connector_PinHeader_2.54mm:PinHeader_1x02_P2.54mm_Vertical, symbol Connector:Conn_01x02_Male
- removed J8: EPWR, Connector_PinHeader_2.54mm:PinHeader_1x02_P2.54mm_Vertical, symbol Connector:Conn_01x02_Male
- removed R1, R10, R2, R3, R33, R34, R35, R36, R37, R38, R39, R4, R40, R5, R6, R7, R8, R9: R, Resistor_SMD:R_0603_1608Metric_Pad0.98x0.95mm_HandSolder, symbol Device:R
- removed R27: 1k, Resistor_SMD:R_0603_1608Metric_Pad0.98x0.95mm_HandSolder, symbol Device:R
- removed R31, R32, R41: 4.7k, Resistor_SMD:R_0603_1608Metric_Pad0.98x0.95mm_HandSolder, symbol Device:R
- removed R43, R44, R45, R46, R47, R48, R49, R50, R51, R52, R53, R54, R55: 1k, Resistor_SMD:R_0402_1005Metric_Pad0.72x0.64mm_HandSolder, symbol Device:R
- removed RP1: Pico_Footprint, CustomFootprints:BluePillModule, symbol custom_symbols:BlackSCSI
- removed U1, U2: SN74CBTD3384, Package_SO:TSSOP-24_4.4x7.8mm_P0.65mm, symbol New_Library:SN74CBTD3384
- removed U3: AMS1117-2.85, Package_TO_SOT_SMD:SOT-223-3_TabPin2, symbol Regulator_Linear:AMS1117CD-2.85
- removed U4, U9: LVT245, Package_SO:TSSOP-20_4.4x6.5mm_P0.65mm, symbol New_Library:LVT245
- removed U5, U6, U7: LVT125, Package_SO:TSSOP-14_4.4x5mm_P0.65mm, symbol New_Library:LVT125
- added C22: 0.1uF, Capacitor_SMD:C_0805_2012Metric_Pad1.18x1.45mm_HandSolder, symbol Device:C
- added C23: 4.7uF, Capacitor_SMD:C_0805_2012Metric_Pad1.18x1.45mm_HandSolder, symbol Device:C
- added D5: D, Diode_SMD:D_SMA, symbol Device:D
- added J10: Conn_01x03_Male, Connector_PinHeader_2.54mm:PinHeader_1x03_P2.54mm_Vertical, symbol Connector:Conn_01x03_Male
- added J11: ACK_En, Connector_PinHeader_2.54mm:PinHeader_1x02_P2.54mm_Vertical, symbol Connector:Conn_01x02_Male
- added J4: USB_C_Receptacle, Connector_USB:USB_C_Receptacle_HRO_TYPE-C-31-M-12, symbol Connector:USB_C_Receptacle
- added J6: SM04B-SRSS-TB(LF)(SN), Library:JST_SM04B-SRSS-TB(LF)(SN), symbol New_Library:SM04B-SRSS-TB(LF)(SN)
- added R61, R65, R66, R67, R68, R69: 1k, Resistor_SMD:R_0402_1005Metric, symbol Device:R
- added RP1: PicoWModule, Library:Raspberry_Pi_PicoW_SMT_THT, symbol New_Library:PicoWModule
- added SD2: MicroSD-TF-06, Library:TF-06_MicroSD, symbol New_Library:MicroSD-TF-06
- added U13, U14, U15, U16: LVT125, Package_SO:TSSOP-14_4.4x5mm_P0.65mm, symbol New_Library:LVT125
- R11: footprint Resistor_SMD:R_0402_1005Metric_Pad0.72x0.64mm_HandSolder -> Resistor_SMD:R_0402_1005Metric
- R20, R21: value 10k -> 5.1k; footprint Resistor_SMD:R_0603_1608Metric_Pad0.98x0.95mm_HandSolder -> Resistor_SMD:R_0402_1005Metric
- R22: value 10k -> 4.7k; footprint Resistor_SMD:R_0603_1608Metric_Pad0.98x0.95mm_HandSolder -> Resistor_SMD:R_0603_1608Metric
- R23, R24, R26: value 1k -> 4.7k; footprint Resistor_SMD:R_0603_1608Metric_Pad0.98x0.95mm_HandSolder -> Resistor_SMD:R_0603_1608Metric
- R25, R28, R29: footprint Resistor_SMD:R_0603_1608Metric_Pad0.98x0.95mm_HandSolder -> Resistor_SMD:R_0402_1005Metric
Connections:
- net +2V8: now also R23.2, U13.14 (Vcc), U14.14 (Vcc), U15.14 (Vcc), U16.14 (Vcc); no longer R20.2, R21.2, R24.2
- net +3V3: now also R24.2, R26.1, C22.2, C23.1, J6.2, RP1.36 (3v3), SD2.4 (VDD)
- net +5VP: now also D5.1 (K), RP1.40 (VBUS_5V)
- net ACK: now also J11.1 (Pin_1), U16.2 (1A)
- net ATN: now also U15.9 (3A)
- net BSY: now also U16.6 (2Y), U16.9 (3A)
- net CD: now also U14.12 (4A), U14.3 (1Y)
- net DBPTr: now also RP1.12 (G9)
- net GND: now also R20.1, R21.1, SW1.1 (2), C22.1, C23.2, J4.A1 (GND), J4.A12 (GND), J4.B1 (GND), J4.B12 (GND), J4.S1 (SHIELD), J6.1, J6.S1 (SHIELD), J6.S2 (SHIELD), RP1.13 (GND), RP1.18 (GND), RP1.23 (GND), RP1.28 (GND), RP1.3 (GND), RP1.33 (A_GND), RP1.38 (GND), RP1.51 (USBGND), RP1.8 (GND), SD2.10 (CASE_GND), SD2.7 (VSS), U13.7 (GND), U14.4 (2/OE), U14.7 (GND), U15.7 (GND), U16.10 (3/OE), U16.7 (GND); no longer R11.1, R23.2, R26.2, SW1.2 (K)
- net IO: now also U13.12 (4A), U13.3 (1Y)
- net MSG: now also U15.12 (4A), U15.3 (1Y)
- net REQ: now also U13.6 (2Y), U13.9 (3A)
- net RST: now also SW1.2 (K), U15.4 (2/OE), U15.5 (2A)
- net SD_CLK: now also RP1.14 (G10), SD2.6 (CLK)
- net SD_CMD_MOSI: now also RP1.15 (G11), SD2.3 (CMD/MOSI)
- net SD_D0_MISO: now also RP1.16 (G12), SD2.8 (DAT0/MISO)
- net SD_D1: now also RP1.17 (G13), SD2.9 (DAT1)
- net SD_D2: now also RP1.19 (G14), SD2.1 (DAT2)
- net SD_D3_CS: now also RP1.20 (G15), SD2.2 (CD/CS/DAT3)
- net SEL: now also U14.5 (2A), U14.8 (3Y)
- net iACK: now also R67.2, U16.3 (1Y)
- net iATN: now also R69.2, U15.8 (3Y)
- net iRST: now also R66.1, U15.6 (2Y)
- net oBSY: now also RP1.32 (G27), U13.1 (1/OE), U13.4 (2/OE), U14.1 (1/OE), U15.1 (1/OE), U15.10 (3/OE), U16.1 (1/OE), U16.4 (2/OE), U16.5 (2A)
- net oCD_iSEL: now also J10.2 (Pin_2), RP1.24 (G18), U14.2 (1A); no longer R28.1
- net oIO: now also R65.2, RP1.29 (G22), U13.2 (1A); no longer R20.1
- net oMSG_iBSY: now also RP1.26 (G20), U15.2 (1A)
- net oREQ: now also R68.1, RP1.25 (G19), U13.5 (2A); no longer R21.1
- net oSEL: now also R66.2, RP1.27 (G21), U14.10 (3/OE), U14.9 (3A)
- net at R42.1: now also RP1.1 (G0)
- net at R13.1: now also RP1.10 (G7)
- net at R12.1: now also RP1.11 (G8)
- net at R19.1: now also RP1.2 (G1)
- net at R18.1: now also RP1.4 (G2)
- net at R17.1: now also RP1.5 (G3)
- net at R16.1: now also RP1.6 (G4)
- net at R15.1: now also RP1.7 (G5)
- net at R14.1: now also RP1.9 (G6)
- net at R11.2: now also J10.3 (Pin_3)
- net BSY_BUFF renamed iBSY
- net iBSY: now also U16.8 (3Y)
- net SEL_BUFF: no longer names the net of R28.2
- net SEL_BUFF: now also J10.1 (Pin_1)
- net oRST renamed SDA
- net SDA: now also J6.3, RP1.21 (G16); no longer SW1.1 (2)
- new net: R61.1, R69.1, RP1.34 (G28)
- new net: J4.B5 (CC2), R21.2
- new net: D5.2 (A), J4.A4 (VBUS), J4.A9 (VBUS), J4.B4 (VBUS), J4.B9 (VBUS)
- new net: J4.A5 (CC1), R20.2
- new net !oBSY: U13.10 (3/OE), U13.13 (4/OE), U14.13 (4/OE), U15.13 (4/OE), U16.13 (4/OE)
- new net ACKDr: J11.2 (Pin_2), U16.11 (4Y)
- new net SCL: J6.4, R26.2, RP1.22 (G17)
- new net USB_DM: J4.A7 (D-), J4.B7 (D-), RP1.52 (USB_DM)
- new net USB_DP: J4.A6 (D+), J4.B6 (D+), RP1.53 (UDB_DP)
- new net iCD: R28.1, U14.11 (4Y)
- new net iIO: R65.1, U13.11 (4Y)
- new net iMSG: R61.2, U15.11 (4Y)
- new net iREQ: R68.2, U13.8 (3Y)
- new net iSEL: R11.1, U14.6 (2Y)
- new net oACK: R67.1, RP1.31 (G26), U16.12 (4A)
Other:
- added sheet Data_Bus_Transceivers_And_Termination (DataBusTransceivers.kicad_sch)
- added sheet SCSI_And_Power (SCSI_And_Power.kicad_sch)
- note added: "BlueSCSI V2, Desktop 50 Pin, Top Connector, 2023.09a"
- note added: "C165948"
- note added: "External I2C "qwiic" by SparkFun"
- note added: "Initiator Mode On Right"
- note added: "PUP Necessary"
- note added: "Raspberry Pi Pico (or W) Stick"
- note added: "SCSI Control Line Bus Buffers"
- note added: "SCSI Signal Order"
- note added: "SD Slot"
- note added: "SM04B-SRSS-TB(LF)(SN) Symbol And Footprint Copyright SnapEDA https://www.snapeda.com/parts/SM04B-SRSS-TB%28LF%29%28SN%29/JST%20Sales/view-part/ License For This Symbol and Footprint Only: CC-BY-SA 4.0 https://creativecommons.org/licenses/by-sa/4.0/ This license contains a warranty disclaimer, please read it in full"
- note added: "Second SD Slot"
- note added: "September 2023"
- note added: "Target Mode On Left"
- note added: "Use Only One SD Slot At A Time! Not Both!"
- note added: "© 2022 - 2023 Tech by Androda, LLC Licensed Attribution-NonCommercial-ShareAlike 4.0 International (CC BY-NC-SA 4.0) https://creativecommons.org/licenses/by-nc-sa/4.0/legalcode"
- note removed: "1k pull resistors Necessary LVT Optional LVTH"
- note removed: "BlueSCSI V2, Desktop 50 Pin, Top Connector, 2023.03a"
- note removed: "March 2023"
- note removed: "Opt. PUP Didn't need them"
- note removed: "RUN is the RP2040 enable pin, and has an internal (on-chip) pull-up resistor to 3.3V of about ~50kΩ. To reset RP2040, short this pin low."
- note removed: "© 2023 Tech by Androda, LLC Licensed Attribution-NonCommercial-ShareAlike 4.0 International (CC BY-NC-SA 4.0) https://creativecommons.org/licenses/by-nc-sa/4.0/legalcode"
- moved on the sheet: H1, H2, H3, R12, R13, R14, R15, R16, R17, R18, R19, R22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

Commit message: Desktop 2023.10a design
Parts:
- removed C23: 4.7uF, Capacitor_SMD:C_0805_2012Metric_Pad1.18x1.45mm_HandSolder, symbol Device:C
- removed D5: D, Diode_SMD:D_SMA, symbol Device:D
- removed J4: USB_C_Receptacle, Connector_USB:USB_C_Receptacle_HRO_TYPE-C-31-M-12, symbol Connector:USB_C_Receptacle
- removed R20, R21: 5.1k, Resistor_SMD:R_0402_1005Metric, symbol Device:R
- removed SD2: MicroSD-TF-06, Library:TF-06_MicroSD, symbol New_Library:MicroSD-TF-06
Other:
- note added: "BlueSCSI V2, Desktop 50 Pin, Top Connector, 2023.10a"
- note added: "October 2023"
- note removed: "BlueSCSI V2, Desktop 50 Pin, Top Connector, 2023.09a"
- note removed: "C165948"
- note removed: "Second SD Slot"
- note removed: "September 2023"
- note removed: "Use Only One SD Slot At A Time! Not Both!"
- moved on the sheet: C22, J6, R24, R26
