File: cc-nc-hardware/Desktop_50_Pin/SCSI_And_Power.kicad_sch (KiCad schematic)
At the start: 19 parts, among them J2 Conn_02x25_Odd_Even, J3 BergFloppy, J7 TERM_BCKF, J8 EPWR, J9 Conn_01x02_Male

Commit message: Desktop 2023.10a design
Parts:
- added C23: 20uF, Capacitor_SMD:C_1206_3216Metric, symbol Device:CP
- added C24: 0.1uF, Capacitor_SMD:C_0805_2012Metric_Pad1.18x1.45mm_HandSolder, symbol Device:C
Connections:
- net +3V3: now also C24.1
- net +5VP: now also C23.1
- net GND: now also C23.2, C24.2
Other:
- note added: "BlueSCSI V2, Desktop 50 Pin, Top Connector, 2023.10a"
- note added: "October 2023"
- note removed: "BlueSCSI V2, Desktop 50 Pin, Top Connector, 2023.09a"
- note removed: "September 2023"
