File: hardware/Centronics_50Pin/Centronics_50Pin.kicad_pcb (KiCad board)
At the start: 2 copper layers, 59.9 x 82.5 mm, 72 parts, among them J2 TRM_BCKF, Q3 AO3401A, U10 Centronics50PinMale, U3 AP1117-ADJ, U4 LVTH245, U5 LVT125, U6 LVT125, U7 LVT125, U8 74HC14, U9 LVTH245

Commit message: Convert BlueSCSI Hardware to CERN OHL-S License (missed a spot)
Other:
- board text removed: "© 2023 Tech by Androda, LLC Licensed Attribution-NonCommercial-ShareAlike 4.0 International (CC BY-NC-SA 4.0) https://creativecommons.org/licenses/by-nc-sa/4.0/legalcode"
Changed lines of the file:
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@@
 		(at 116.6876 106.3244 180)
 		(property "Reference" "G***"
-			(at 0 0 360)
+			(at 0 0 0)
 			(layer "B.SilkS")
 			(hide yes)
@@
 		)
 		(property "Value" "LOGO"
-			(at 0.75 0 360)
+			(at 0.75 0 0)
 			(layer "B.SilkS")
 			(hide yes)
@@
 		)
 		(property "Footprint" ""
-			(at 0 0 360)
+			(at 0 0 0)
 			(layer "B.Fab")
 			(hide yes)
@@
 		)
 		(property "Datasheet" ""
-			(at 0 0 360)
+			(at 0 0 0)
 			(layer "B.Fab")
 			(hide yes)
@@
 		)
 		(property "Description" ""
-			(at 0 0 360)
+			(at 0 0 0)
 			(layer "B.Fab")
 			(hide yes)
@@
 		)
 	)
-	(gr_text "© 2023 Tech by Androda, LLC\nLicensed Attribution-NonCommercial-ShareAlike 4.0 International (CC BY-NC-SA 4.0)\nhttps://creativecommons.org/licenses/by-nc-sa/4.0/legalcode"
-		(at 180.75 174.18 0)
-		(layer "Cmts.User")
-		(effects
-			(font
-				(size 1 1)
-				(thickness 0.15)
-			)
-			(justify left bottom)
-		)
-	)
