File: hardware/USB_Bridge/Desktop_50_Pin_TopConn.kicad_pcb (KiCad board)
At the start: 4 copper layers, 50 x 40 mm, 154 parts, among them J1 ACK_En, J10 BergFloppy, J12 USB_C_Receptacle_USB2.0, J13 Conn_01x03_Male, J14 Debug, J3 DB25_Plug_MountingHoles, J4 SM04B-SRSS-TB(LF)(SN), J5 Conn_01x03_Male, J6 Conn_01x03_Male, J7 TERM_BCKF, J8 EPWR, Q1 AO3401A, Q2 AO3401A, Q3 DMG1012T, SW1 SCSI Reset, SW2 USB Boot, SW3 RP2040 Reset, U1 LVT125, U10 AMS1117-2.85, U11 AMS1117-3.3, U12 W25Q16JVUXIQ, U13 RP2040, U2 LVT125, U3 LVT125, U4 LVT125, U5 74HC14, U6 LVT245, U7 LVT245, U8 LVT245, U9 LVT245, Y1 12MHz

Commit message: more routing fun....
Parts:
- removed TP1: TestPoint_Small, TestPoint:TestPoint_Pad_D1.0mm
- J14, J5: footprint Connector_PinHeader_2.54mm:PinHeader_1x03_P2.54mm_Vertical -> Connector_PinHeader_2.54mm:PinHeader_1x03_P2.54mm_Vertical_SMD_Pin1Left; moved to B.Cu
- JP1: moved to B.Cu
- SD1: moved to F.Cu
- moved SW1 50.0 mm to (111.4, 117.0), turned to 0 degrees
- moved SD1 46.0 mm to (158.3, 96.7), turned to -90 degrees
- moved SW3 44.7 mm to (154.9, 117.0), turned to 0 degrees
- moved R2 42.4 mm to (134.1, 113.9), turned to 90 degrees
- moved C40 41.6 mm to (134.0, 112.1), turned to 180 degrees
- moved C5 40.1 mm to (116.5, 87.0), turned to 0 degrees
- moved R46 39.9 mm to (117.1, 85.7), turned to 180 degrees
- moved C16 38.0 mm to (117.8, 95.8), turned to 0 degrees
- moved SW2 34.5 mm to (160.0, 99.8), turned to 180 degrees
- moved C42 34.1 mm to (134.1, 106.3)
- moved R26 33.4 mm to (125.0, 95.0)
- moved R27 31.8 mm to (125.0, 93.8), turned to 180 degrees
- moved C4 30.2 mm to (116.5, 113.1)
- moved J5 28.4 mm to (131.8, 95.0), turned to 180 degrees
- moved J4 28.1 mm to (152.7, 115.1), turned to 0 degrees
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Routing:
- net GND: track 125.5 -> 225.2 mm, vias 43 -> 61
- net oBSY: track 0.00 -> 79.9 mm, vias 0 -> 11
- net +3V3: track 0.00 -> 60.8 mm, vias 0 -> 16
- net oREQ: track 0.00 -> 47.8 mm, vias 0 -> 3
- net oIO: track 0.00 -> 45.0 mm, vias 0 -> 3
- net oSEL: track 0.00 -> 44.1 mm, vias 0 -> 3
- net !oBSY: track 0.00 -> 42.9 mm, vias 0 -> 6
- net oCD_iSEL: track 0.00 -> 39.4 mm, vias 0 -> 3
- net oACK: track 0.00 -> 38.1 mm, vias 0 -> 3
- net oMSG_iBSY: track 0.00 -> 36.7 mm, vias 0 -> 3
- net SD_D0_MISO: track 0.00 -> 35.3 mm, vias 0 -> 2
- net Net-(D1-A): track 0.00 -> 34.3 mm, vias 0 -> 2
- net CD: track 35.0 -> 2.17 mm, vias 3 -> 2
- net /Pico/GPIO28: track 0.00 -> 31.5 mm, vias 0 -> 3
- net /Pico/RUN: track 0.00 -> 31.0 mm, vias 0 -> 4
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- added copper zone on In1.Cu, net +3V3
Other:
- board size 50 x 40 mm -> 65 x 40 mm

Commit message: as-ordered PROTOTYPE
Parts:
- removed C41: 1n 25V, Capacitor_SMD:C_0402_1005Metric
- removed D5: Schottky Diode, Diode_SMD:D_SOD-123
- removed F2: Polyfuse, Fuse:Fuse_0805_2012Metric_Pad1.15x1.40mm_HandSolder
- removed J7: TERM_BCKF, Jumper:SolderJumper-2_P1.3mm_Open_RoundedPad1.0x1.5mm
- removed J8: EPWR, Jumper:SolderJumper-2_P1.3mm_Open_RoundedPad1.0x1.5mm
- removed Q3: DMG1012T, Package_TO_SOT_SMD:SOT-523
- removed R59: 200k, Resistor_SMD:R_0402_1005Metric
- removed R60: 100k, Resistor_SMD:R_0402_1005Metric
- added C43: 0.1uF, Capacitor_SMD:C_0402_1005Metric, F.Cu at (144.6, 97.2)
- added D8: Schottky Diode, Diode_SMD:D_SOD-123, F.Cu at (147.8, 97.3)
- added D9: Schottky Diode, Diode_SMD:D_SOD-123, F.Cu at (147.8, 92.2)
- added F3: Polyfuse, Fuse:Fuse_0805_2012Metric_Pad1.15x1.40mm_HandSolder, F.Cu at (154.4, 105.4)
- added F4: Polyfuse, Fuse:Fuse_0805_2012Metric_Pad1.15x1.40mm_HandSolder, F.Cu at (146.3, 86.4)
- added F5: Polyfuse, Fuse:Fuse_0805_2012Metric_Pad1.15x1.40mm_HandSolder, F.Cu at (143.5, 93.0)
- added JP3: USB Pwr En, Jumper:SolderJumper-2_P1.3mm_Open_TrianglePad1.0x1.5mm, B.Cu at (148.3, 99.1)
- added JP4: Berg Pwr En, Jumper:SolderJumper-2_P1.3mm_Open_TrianglePad1.0x1.5mm, B.Cu at (148.3, 93.0)
- added JP5: Term Input Pwr En, Jumper:SolderJumper-2_P1.3mm_Open_TrianglePad1.0x1.5mm, B.Cu at (148.3, 96.0)
- added JP6: Term Output En, Jumper:SolderJumper-2_P1.3mm_Open_TrianglePad1.0x1.5mm, B.Cu at (138.9, 94.7)
- added JP7: USB Bridge En, Jumper:SolderJumper-3_P1.3mm_Open_RoundedPad1.0x1.5mm, B.Cu at (146.0, 115.0)
- added R3: 1k, Resistor_SMD:R_0402_1005Metric, F.Cu at (147.8, 113.2)
- added R4: 1k, Resistor_SMD:R_0402_1005Metric, F.Cu at (147.8, 112.2)
- C19, C20, C24: value 4.7uF -> 25V 10uF
- C21: value 4.7uF -> 0.1uF; footprint Capacitor_SMD:C_0603_1608Metric -> Capacitor_SMD:C_0402_1005Metric
- C22, C8: value 20uF -> 4.7uF
- C25, C26: value 10u 6.3V -> 25V 10uF; footprint Capacitor_SMD:C_0402_1005Metric -> Capacitor_SMD:C_0603_1608Metric
- C9: value 20uF -> 25V 10uF
- D4: value Schottky Diode -> Schottky
- G***: moved to F.Cu
- J3: value DB25_Plug_MountingHoles -> SCSI Connector
- moved G*** 31.2 mm to (152.7, 117.1), turned to 0 degrees
- moved C24 26.3 mm to (117.9, 99.8), turned to 0 degrees
- moved C21 18.5 mm to (128.3, 95.5)
- moved R49 15.6 mm to (153.4, 107.0), turned to 180 degrees
- moved C23 13.8 mm to (133.6, 92.3), turned to 0 degrees
- moved J13 12.9 mm to (131.8, 93.2)
- moved R51 12.1 mm to (151.4, 107.0), turned to 180 degrees
- moved C20 11.6 mm to (136.2, 91.7)
- moved U11 9.83 mm to (135.1, 96.5), turned to 180 degrees
- moved C22 9.80 mm to (140.5, 94.2), turned to 90 degrees
- moved D4 7.91 mm to (147.8, 89.7)
- moved C19 7.51 mm to (139.4, 91.7)
- moved C26 7.03 mm to (141.9, 97.8), turned to -90 degrees
- moved J5 5.71 mm to (134.9, 99.8), turned to 90 degrees
- moved C17 4.55 mm to (143.4, 97.8), turned to -90 degrees
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Connections:
- C11 pad 1: +5F -> +5V
- C12 pad 1: +5F -> +5V
- C20 pad 1: Net-(D3-K) -> +5V
- C21 pad 1: +5VP -> +5V
- C22 pad 1: +5VP -> +5V
- C23 pad 2: +5F -> +5V
- C24 pad 1: +5F -> +2V8
- C25 pad 1: GND -> +3V3
- C25 pad 2: /Pico/VSYS -> GND
- C8 pad 1: +5F -> +5V
- D3 pad 2: +5V -> Net-(D3-A)
- D4 pad 1: Net-(D3-K) -> Net-(D4-K)
- F1 pad 1: Net-(D3-K) -> EXT_TERM_PWR
- F1 pad 2: Net-(J7-Pin_2) -> Net-(D3-K)
- J10 pad 1: Net-(D4-A) -> Net-(J10-5V)
- J3 pad 25: +5V -> EXT_TERM_PWR
- U10 pad 3: +5F -> +5V
- U11 pad 3: /Pico/VSYS -> +5V
- U5 pad 13: +5F -> +5V
- U5 pad 14: +5F -> +5V
Routing:
- net GND: track 225.2 -> 329.2 mm, vias 61 -> 95
- net +5V: track 3.32 -> 70.1 mm, vias 2 -> 4
- net EXT_TERM_PWR: track 0.00 -> 59.4 mm, vias 0 -> 3
- net CD: track 2.17 -> 43.4 mm, vias 2 -> 4
- net ATN: track 8.92 -> 49.5 mm, vias 3 -> 6
- net SD_CMD_MOSI: track 0.00 -> 36.7 mm, vias 0 -> 2
- net SD_CLK: track 0.00 -> 33.9 mm, vias 0 -> 2
- net +2V8: track 79.4 -> 110.4 mm
- net RST: track 41.4 -> 70.8 mm, vias 4 -> 6
- net +3V3: track 60.8 -> 89.2 mm
- net TRM_ON_J: track 31.3 -> 55.9 mm, vias 1 -> 3
- net SD_D2: track 17.8 -> 39.9 mm, vias 1 -> 2
- net SD_D3_CS: track 12.9 -> 34.7 mm, vias 1 -> 2
- net iBSY: track 0.00 -> 19.7 mm, vias 0 -> 2
- net VBUS: track 0.00 -> 13.7 mm
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Other:
- board text added: "150"
- board text added: "330"
- board text added: "ACK"
- board text added: "ATN"
- board text added: "BAD WOLF"
- board text added: "BERG"
- board text added: "BOOT SEL"
- board text added: "BSY"
- board text added: "BlueSCSI v2"
- board text added: "CD"
- board text added: "DB0"
- board text added: "DB1"
- board text added: "DB2"
- board text added: "DB3"
- board text added: "DB4"
- board text added: "DB5"
- board text added: "DB6"
- board text added: "DB7"
- board text added: "DBP"
- board text added: "DIO"
- board text added: "DIS"
- board text added: "Debug"
- board text added: "EN"
- board text added: "EXT LED"
- board text added: "Enable ONE Power Input"
- board text added: "GND"
- board text added: "GP23"
- board text added: "GP25"
- board text added: "INIT"
- board text added: "INITIATOR OR TARGET"
- board text added: "IO"
- board text added: "LED BRIGHT"
- board text added: "MSG"
- board text added: "Mode Sel"
- board text added: "POWER INPUT"
- board text added: "PROTOTYPE"
- board text added: "REQ"
- board text added: "RESET MCU"
- board text added: "RST"
- board text added: "SCSI RESET"
- board text added: "SD Card Mode"
- board text added: "SEL"
- board text added: "TARGET"
- board text added: "TERM"
- board text added: "TERM Backfeed"
- board text added: "TERM PWR OUT"
- board text added: "TRM PWR OUTPUT"
- board text added: "USB"
- board text added: "USB Bridge"
- board text added: "github.com/BlueSCSI/BlueSCSI-v2 BlueSCSI © Eric Helgeson PCB © akuker and Tech by Androda, LLC"
- board text removed: "110_T"
- board text removed: "18 scsi signals"
- board text removed: "BACK"
- board text removed: "FEED"
- board text removed: "Initiator"
- board text removed: "LED"
- board text removed: "Manufactured By:"
- board text removed: "PWR_ON"
- board text removed: "TRM_OFF"
- board text removed: "TRM_ON"
- board text removed: "Target"
- board text removed: "github.com/BlueSCSI/BlueSCSI-v2 BlueSCSI © Eric Helgeson PCB © Tech by Androda, LLC"
