File: hardware/USB_Bridge/Desktop_50_Pin_TopConn.kicad_sch (KiCad schematic)
At the start: 37 parts, among them J10 Conn_01x03_Male, J11 ACK_En, J6 SM04B-SRSS-TB(LF)(SN), SW1 SW_MEC_5E, U13 LVT125, U14 LVT125, U15 LVT125, U16 LVT125

Commit message: intermediate checkin
Parts:
- C1: renamed from C22; footprint Capacitor_SMD:C_0805_2012Metric_Pad1.18x1.45mm_HandSolder -> Capacitor_SMD:C_0805_2012Metric
- J1: renamed from J11; footprint Connector_PinHeader_2.54mm:PinHeader_1x02_P2.54mm_Vertical -> Jumper:SolderJumper-2_P1.3mm_Open_RoundedPad1.0x1.5mm
- J2: renamed from J10; footprint Connector_PinHeader_2.54mm:PinHeader_1x03_P2.54mm_Vertical -> Jumper:SolderJumper-3_P1.3mm_Open_RoundedPad1.0x1.5mm
- J4: renamed from J6; MP SM04B-SRSS-TB(LF)(SN) -> (none); STANDARD Manufacturer recommendations -> (none)
- R10: renamed from R12; footprint Resistor_SMD:R_0402_1005Metric_Pad0.72x0.64mm_HandSolder -> Resistor_SMD:R_0402_1005Metric
- R12: renamed from R13; footprint Resistor_SMD:R_0402_1005Metric_Pad0.72x0.64mm_HandSolder -> Resistor_SMD:R_0402_1005Metric
- R13: renamed from R14; footprint Resistor_SMD:R_0402_1005Metric_Pad0.72x0.64mm_HandSolder -> Resistor_SMD:R_0402_1005Metric
- R14: renamed from R15; footprint Resistor_SMD:R_0402_1005Metric_Pad0.72x0.64mm_HandSolder -> Resistor_SMD:R_0402_1005Metric
- R16, R17, R18: footprint Resistor_SMD:R_0402_1005Metric_Pad0.72x0.64mm_HandSolder -> Resistor_SMD:R_0402_1005Metric
- R20: renamed from R19; footprint Resistor_SMD:R_0402_1005Metric_Pad0.72x0.64mm_HandSolder -> Resistor_SMD:R_0402_1005Metric
- R21: renamed from R42; footprint Resistor_SMD:R_0402_1005Metric_Pad0.72x0.64mm_HandSolder -> Resistor_SMD:R_0402_1005Metric
- RP1: footprint Library:Raspberry_Pi_PicoW_SMT_THT -> Library:Raspberry_Pi_PicoW_SMT_Only
- U1: renamed from U13; footprint Package_SO:TSSOP-14_4.4x5mm_P0.65mm -> Package_SO:SO-14_3.9x8.65mm_P1.27mm; LCSC (none) -> C548964
- U2: renamed from U14; footprint Package_SO:TSSOP-14_4.4x5mm_P0.65mm -> Package_SO:SO-14_3.9x8.65mm_P1.27mm; LCSC (none) -> C548964
- U3: renamed from U15; footprint Package_SO:TSSOP-14_4.4x5mm_P0.65mm -> Package_SO:SO-14_3.9x8.65mm_P1.27mm; LCSC (none) -> C548964
- U4: renamed from U16; footprint Package_SO:TSSOP-14_4.4x5mm_P0.65mm -> Package_SO:SO-14_3.9x8.65mm_P1.27mm; LCSC (none) -> C548964
- renumbered H3 to H1, H1 to H3, R11 to R1, R67 to R11, R69 to R15, R61 to R19, R28 to R2, R24 to R22, R26 to R23, R68 to R3, R29 to R4, R22 to R5, R66 to R6, R23 to R7, R65 to R8, R25 to R9
Other:
- added sheet piccolo (piccolo.kicad_sch)

Commit message: intermediate - horizonal r's
Parts:
- removed J2: Conn_01x03_Male, Jumper:SolderJumper-3_P1.3mm_Open_RoundedPad1.0x1.5mm, symbol Connector:Conn_01x03_Male
- removed R1, R10, R11, R12, R13, R14, R15, R16, R17, R18, R19, R2, R20, R21, R3, R4, R6, R8: 1k, Resistor_SMD:R_0402_1005Metric, symbol Device:R
- removed RP1: PicoWModule, Library:Raspberry_Pi_PicoW_SMT_Only, symbol New_Library:PicoWModule
Connections:
- no-connect marks 0 -> 13
Other:
- note removed: "Raspberry Pi Pico (or W) Stick"
- note removed: "Series current-limiter Necessary for LVT and LVTH"
- moved on the sheet: C1, J4, R22, R23, R5, R7, R9, SD1, SW1

Commit message: initial rough parts placement
Parts:
- SD1: footprint CustomFootprints:SOFNG_SD-001 -> Connector_Card:microSD_HC_Molex_104031-0811; LCSC (none) -> C2982548
Changed lines of the file:
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@@
 			)
 		)
-		(property "Footprint" "CustomFootprints:SOFNG_SD-001"
+		(property "Footprint" "Connector_Card:microSD_HC_Molex_104031-0811"
 			(at 39.37 93.98 0)
 			(effects
@@
 			(at 39.37 99.06 0)
 			(effects
+				(font
+					(size 1.27 1.27)
+				)
+				(hide yes)
+			)
+		)
+		(property "LCSC" "C2982548"
+			(at 39.37 99.06 0)
+			(effects

Commit message: more routing
Parts:
- removed SD1: SOFNG_SD-001, Connector_Card:microSD_HC_Molex_104031-0811, symbol custom_symbols:SOFNG_SD-001
- added H4: MountingHole, MountingHole:MountingHole_2.2mm_M2, symbol Mechanical:MountingHole
- C1: footprint Capacitor_SMD:C_0805_2012Metric -> Capacitor_SMD:C_0402_1005Metric; LCSC (none) -> C307331
- H1, H2, H3: footprint MountingHole:MountingHole_3.2mm_M3 -> MountingHole:MountingHole_2.2mm_M2; LCSC (none) -> --
- J1: LCSC (none) -> --
- J4: LCSC (none) -> C160404
- R22, R23, R5, R7: LCSC (none) -> C23162
- R9: LCSC (none) -> C11702
- SW1: value SW_MEC_5E -> SCSI Reset; footprint Library:TS-1187A-B-A-B -> Button_Switch_SMD:SW_Push_1P1T_XKB_TS-1187A; symbol Switch:SW_MEC_5E -> Switch:SW_Push; LCSC (none) -> C318884
- U1, U2, U3, U4: footprint Package_SO:SO-14_3.9x8.65mm_P1.27mm -> Package_SO:TSSOP-14_4.4x5mm_P0.65mm; LCSC C548964 -> C2675577
Connections:
- no-connect marks 13 -> 9
Other:
- sheet piccolo renamed Pico
- note removed: "SD Slot"
- moved on the sheet: R5, R7, R9

Commit message: as-ordered PROTOTYPE
Parts:
- C1: symbol Device:C -> Device:C_Small
Other:
- moved on the sheet: C1
Changed lines of the file:
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@@
+		)
+	)
+	(wire
+		(pts
+			(xy 25.4 166.37) (xy 32.385 166.37)
+		)
+		(stroke
+			(width 0)
+			(type default)
 		)
 	)
@@
 		)
 	)
-	(wire
+	(polyline
 		(pts
-			(xy 26.035 166.37) (xy 32.385 166.37)
+			(xy 17.78 183.515) (xy 17.78 151.765)
 		)
 		(stroke
@@
 	(polyline
 		(pts
-			(xy 17.78 183.515) (xy 17.78 151.765)
+			(xy 285.115 50.8) (xy 95.25 50.8)
 		)
 		(stroke
@@
 	(polyline
 		(pts
-			(xy 285.115 50.8) (xy 95.25 50.8)
+			(xy 93.345 49.53) (xy 93.345 13.97)
 		)
 		(stroke
@@
 	(polyline
 		(pts
-			(xy 93.345 49.53) (xy 93.345 13.97)
+			(xy 84.455 13.97) (xy 84.455 49.53)
 		)
 		(stroke
@@
 	(polyline
 		(pts
-			(xy 84.455 13.97) (xy 84.455 49.53)
+			(xy 95.25 13.335) (xy 285.115 13.335)
 		)
 		(stroke
@@
 		)
 	)
-	(polyline
+	(wire
 		(pts
-			(xy 95.25 13.335) (xy 285.115 13.335)
+			(xy 32.385 166.37) (xy 33.655 166.37)
 		)
 		(stroke
@@
 	(wire
 		(pts
-			(xy 32.385 166.37) (xy 33.655 166.37)
+			(xy 25.4 172.72) (xy 25.4 173.99)
 		)
 		(stroke
@@
 		(pts
 			(xy 285.115 13.335) (xy 285.115 50.8)
+		)
+		(stroke
+			(width 0)
+			(type default)
+		)
+	)
+	(wire
+		(pts
+			(xy 25.4 167.64) (xy 25.4 166.37)
 		)
 		(stroke
@@
 	)
 	(symbol
-		(lib_id "Device:C")
-		(at 26.035 170.18 180)
+		(lib_id "Device:C_Small")
+		(at 25.4 170.18 180)
 		(unit 1)
 		(exclude_from_sim no)
@@
 		(dnp no)
 		(property "Reference" "C1"
-			(at 19.6342 170.18 90)
+			(at 18.9992 170.18 90)
 			(effects
 				(font
@@
 		)
 		(property "Value" "0.1uF"
-			(at 21.9456 170.18 90)
+			(at 21.3106 170.18 90)
 			(effects
 				(font
@@
 		)
 		(property "Footprint" "Capacitor_SMD:C_0402_1005Metric"
-			(at 25.0698 166.37 0)
+			(at 25.4 170.18 0)
 			(effects
 				(font
@@
 		)
 		(property "Datasheet" "~"
-			(at 26.035 170.18 0)
-			(effects
-				(font
-					(size 1.27 1.27)
-				)
-				(hide yes)
-			)
-		)
-		(property "Description" ""
-			(at 26.035 170.18 0)
+			(at 25.4 170.18 0)
+			(effects
+				(font
+					(size 1.27 1.27)
+				)
+				(hide yes)
+			)
+		)
+		(property "Description" "Unpolarized capacitor, small symbol"
+			(at 25.4 170.18 0)
 			(effects
 				(font
@@
 		)
 		(property "LCSC" "C307331"
-			(at 26.035 170.18 0)
+			(at 25.4 170.18 0)
 			(effects
 				(font
@@
 	(symbol
 		(lib_id "power:GND")
-		(at 26.035 173.99 0)
+		(at 25.4 173.99 0)
 		(mirror y)
 		(unit 1)
@@
 		(dnp no)
 		(property "Reference" "#PWR034"
-			(at 26.035 180.34 0)
+			(at 25.4 180.34 0)
 			(effects
 				(font
@@
 		)
 		(property "Value" "GND"
-			(at 25.908 178.3842 90)
+			(at 25.273 178.3842 90)
 			(effects
 				(font
@@
 		)
 		(property "Footprint" ""
-			(at 26.035 173.99 0)
+			(at 25.4 173.99 0)
 			(effects
 				(font
@@
 		)
 		(property "Datasheet" ""
-			(at 26.035 173.99 0)
+			(at 25.4 173.99 0)
 			(effects
 				(font
@@
 		)
 		(property "Description" ""
-			(at 26.035 173.99 0)
-			(effects
-				(font
+			(at 25.4 173.99 0)
+			(effects
+				(font
