File: hardware/USB_Bridge/LED_Indicators.kicad_sch (KiCad schematic)
At the start: 10 parts, among them J5 Conn_01x03_Male, U8 74HC14

Commit message: intermediate checkin
Parts:
- D1: renamed from D3; JLCPCB Part Number C72041 -> (none)
- D2: renamed from D4; JLCPCB Part # C2290 -> (none)
- R25: renamed from R56; footprint Resistor_SMD:R_0603_1608Metric_Pad0.98x0.95mm_HandSolder -> Resistor_SMD:R_0603_1608Metric
- U5: renamed from U8; footprint (none) -> Package_SO:SOIC-14_3.9x8.7mm_P1.27mm; LCSC (none) -> C5605
- U5: renamed from U8; footprint Package_SO:SO-14_3.9x8.65mm_P1.27mm -> Package_SO:SOIC-14_3.9x8.7mm_P1.27mm; JLC Part # C5605 -> (none); LCSC (none) -> C5605
- renumbered JP2 to JP1, JP1 to JP2, R30 to R24, R58 to R26, R59 to R27

Commit message: intermediate - horizonal r's
Connections:
- no-connect marks 0 -> 1
Other:
- moved on the sheet: D1, D2, J5, JP1, JP2, R24, R25, R26, R27, U5A, U5B, U5C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

Commit message: initial rough parts placement
Parts:
- R24: footprint Resistor_SMD:R_0402_1005Metric_Pad0.72x0.64mm_HandSolder -> Resistor_SMD:R_0402_1005Metric
- R26, R27: footprint Resistor_SMD:R_0603_1608Metric_Pad0.98x0.95mm_HandSolder -> Resistor_SMD:R_0402_1005Metric
Changed lines of the file:
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@@
 			)
 		)
-		(property "Footprint" "Resistor_SMD:R_0603_1608Metric_Pad0.98x0.95mm_HandSolder"
+		(property "Footprint" "Resistor_SMD:R_0402_1005Metric"
 			(at 144.78 117.348 90)
 			(effects
@@
 			)
 		)
-		(property "Footprint" "Resistor_SMD:R_0603_1608Metric_Pad0.98x0.95mm_HandSolder"
+		(property "Footprint" "Resistor_SMD:R_0402_1005Metric"
 			(at 137.16 117.348 90)
 			(effects
@@
 			)
 		)
-		(property "Footprint" "Resistor_SMD:R_0402_1005Metric_Pad0.72x0.64mm_HandSolder"
+		(property "Footprint" "Resistor_SMD:R_0402_1005Metric"
 			(at 145.415 69.723 90)
 			(effects

Commit message: more routing
Parts:
- D1, D2: footprint LED_SMD:LED_0603_1608Metric_Pad1.05x0.95mm_HandSolder -> LED_SMD:LED_0805_2012Metric; LCSC (none) -> C2297
- J5, JP1, JP2: LCSC (none) -> --
- R24: LCSC (none) -> C25117
- R25: LCSC (none) -> C23162
- R26: LCSC (none) -> C25082
- R27: LCSC (none) -> C25104
- U5: footprint Package_SO:SOIC-14_3.9x8.7mm_P1.27mm -> Package_SO:TSSOP-14_4.4x5mm_P0.65mm; LCSC C5605 -> C6821
Changed lines of the file:
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@@
+			)
+		)
+		(property "LCSC" "C25104"
+			(at 144.78 115.57 0)
+			(effects
+				(font
+					(size 1.27 1.27)
+				)
+				(hide yes)
 			)
 		)
@@
 			)
 		)
+		(property "LCSC" "C25082"
+			(at 137.16 115.57 0)
+			(effects
+				(font
+					(size 1.27 1.27)
+				)
+				(hide yes)
+			)
+		)
 		(pin "1"
 		)
@@
 			)
 		)
-		(property "Footprint" "Package_SO:SOIC-14_3.9x8.7mm_P1.27mm"
+		(property "Footprint" "Package_SO:TSSOP-14_4.4x5mm_P0.65mm"
 			(at 133.985 67.945 0)
 			(effects
@@
 			)
 		)
-		(property "LCSC" "C5605"
+		(property "LCSC" "C6821"
 			(at 133.985 67.945 0)
 			(effects
@@
 			)
 		)
-		(property "Footprint" "Package_SO:SOIC-14_3.9x8.7mm_P1.27mm"
+		(property "Footprint" "Package_SO:TSSOP-14_4.4x5mm_P0.65mm"
 			(at 163.83 146.05 0)
 			(effects
@@
 			)
 		)
-		(property "LCSC" "C5605"
+		(property "LCSC" "C6821"
 			(at 163.83 146.05 0)
 			(effects
@@
 			)
 		)
+		(property "LCSC" "--"
+			(at 137.16 121.92 0)
+			(effects
+				(font
+					(size 1.27 1.27)
+				)
+				(hide yes)
+			)
+		)
 		(pin "1"
 		)
@@
 			)
 		)
+		(property "LCSC" "--"
+			(at 144.78 107.95 0)
+			(effects
+				(font
+					(size 1.27 1.27)
+				)
+				(hide yes)
+			)
+		)
 		(pin "1"
 		)
@@
 			)
 		)
-		(property "Footprint" "Package_SO:SOIC-14_3.9x8.7mm_P1.27mm"
+		(property "Footprint" "Package_SO:TSSOP-14_4.4x5mm_P0.65mm"
 			(at 125.73 90.17 0)
 			(effects
@@
 			)
 		)
-		(property "LCSC" "C5605"
+		(property "LCSC" "C6821"
 			(at 125.73 90.17 0)
 			(effects
@@
 			)
 		)
+		(property "LCSC" "C23162"
+			(at 152.4 90.17 0)
+			(effects
+				(font
+					(size 1.27 1.27)
+				)
+				(hide yes)
+			)
+		)
 		(pin "1"
 		)
@@
 			)
 		)
-		(property "Footprint" "Package_SO:SOIC-14_3.9x8.7mm_P1.27mm"
+		(property "Footprint" "Package_SO:TSSOP-14_4.4x5mm_P0.65mm"
 			(at 123.19 115.57 0)
 			(effects
@@
 			)
 		)
-		(property "LCSC" "C5605"
+		(property "LCSC" "C6821"
 			(at 123.19 115.57 0)
 			(effects
@@
 			)
 		)
-		(property "Footprint" "Package_SO:SOIC-14_3.9x8.7mm_P1.27mm"
+		(property "Footprint" "Package_SO:TSSOP-14_4.4x5mm_P0.65mm"
 			(at 140.97 38.1 0)
 			(effects
@@
 			)
 		)
-		(property "LCSC" "C5605"
+		(property "LCSC" "C6821"
 			(at 140.97 38.1 0)
 			(effects
@@
 			)
 		)
-		(property "Footprint" "LED_SMD:LED_0603_1608Metric_Pad1.05x0.95mm_HandSolder"
+		(property "Footprint" "LED_SMD:LED_0805_2012Metric"
 			(at 153.035 67.945 0)
 			(effects
@@
 		)
 		(property "Description" ""
+			(at 153.035 67.945 0)
+			(effects
+				(font
+					(size 1.27 1.27)
+				)
+				(hide yes)
+			)
+		)
+		(property "LCSC" "C2297"
 			(at 153.035 67.945 0)
 			(effects
@@
 			)
 		)
-		(property "Footprint" "Package_SO:SOIC-14_3.9x8.7mm_P1.27mm"
+		(property "Footprint" "Package_SO:TSSOP-14_4.4x5mm_P0.65mm"
 			(at 119.38 146.685 0)
 			(effects
@@
 			)
 		)
-		(property "LCSC" "C5605"
+		(property "LCSC" "C6821"
 			(at 119.38 146.685 0)
 			(effects
@@
 			)
 		)
-		(property "Footprint" "LED_SMD:LED_0603_1608Metric_Pad1.05x0.95mm_HandSolder"
+		(property "Footprint" "LED_SMD:LED_0805_2012Metric"
 			(at 160.02 90.17 0)
 			(effects
@@
 		)
 		(property "Description" ""
+			(at 160.02 90.17 0)
+			(effects
+				(font
+					(size 1.27 1.27)
+				)
+				(hide yes)
+			)
+		)
+		(property "LCSC" "C2297"
 			(at 160.02 90.17 0)
 			(effects
@@
 			)
 		)
+		(property "LCSC" "C25117"
+			(at 145.415 67.945 0)
+			(effects
+				(font
+					(size 1.27 1.27)
+				)
+				(hide yes)
+			)
+		)
 		(pin "1"
 		)
@@
 			)
 		)
+		(property "LCSC" "--"
+			(at 172.72 115.57 0)
+			(effects
+				(font
+					(size 1.27 1.27)
+				)
+				(hide yes)
+			)
+		)
 		(pin "1"
 		)
@@
 			)
 		)
-		(property "Footprint" "Package_SO:SOIC-14_3.9x8.7mm_P1.27mm"
+		(property "Footprint" "Package_SO:TSSOP-14_4.4x5mm_P0.65mm"
 			(at 140.97 90.17 0)
 			(effects
@@
 			)
 		)
-		(property "LCSC" "C5605"
+		(property "LCSC" "C6821"
 			(at 140.97 90.17 0)
 			(effects

Commit message: more routing fun....
Parts:
- J5: footprint Connector_PinHeader_2.54mm:PinHeader_1x03_P2.54mm_Vertical -> Connector_PinHeader_2.54mm:PinHeader_1x03_P2.54mm_Vertical_SMD_Pin1Left
Changed lines of the file:
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@@
 			)
 		)
-		(property "Footprint" "Connector_PinHeader_2.54mm:PinHeader_1x03_P2.54mm_Vertical"
+		(property "Footprint" "Connector_PinHeader_2.54mm:PinHeader_1x03_P2.54mm_Vertical_SMD_Pin1Left"
 			(at 172.72 115.57 0)
 			(effects

Commit message: as-ordered PROTOTYPE
Parts:
- added C21: 0.1uF, Capacitor_SMD:C_0402_1005Metric, symbol Device:C_Small
Connections:
- net GND: now also C21.2
- net +5F renamed +5V
- net +5V: now also C21.1
