File: hardware/USB_Bridge/SCSI_And_Power.kicad_sch (KiCad schematic)
At the start: 21 parts, among them J2 Conn_02x25_Odd_Even, J3 BergFloppy, J7 TERM_BCKF, J8 EPWR, J9 Conn_01x02_Male

Commit message: intermediate checkin
Parts:
- removed J2: Conn_02x25_Odd_Even, Connector_PinHeader_2.54mm:PinHeader_2x25_P2.54mm_Horizontal, symbol Connector_Generic:Conn_02x25_Odd_Even
- added J3: DB25_Plug_MountingHoles, Connector_Dsub:DSUB-25_Male_Horizontal_P2.77x2.84mm_EdgePinOffset4.94mm_Housed_MountingHolesOffset7.48mm, symbol Connector:DB25_Plug_MountingHoles
- C13: renamed from C19; footprint Capacitor_SMD:C_0805_2012Metric_Pad1.18x1.45mm_HandSolder -> Capacitor_SMD:C_0805_2012Metric
- C14: renamed from C9; footprint Capacitor_SMD:C_0805_2012Metric_Pad1.18x1.45mm_HandSolder -> Capacitor_SMD:C_0805_2012Metric
- C15: renamed from C13; footprint Capacitor_SMD:C_0805_2012Metric_Pad1.18x1.45mm_HandSolder -> Capacitor_SMD:C_0805_2012Metric
- C16: renamed from C14; footprint Capacitor_SMD:C_0805_2012Metric_Pad1.18x1.45mm_HandSolder -> Capacitor_SMD:C_0805_2012Metric
- C17: renamed from C12; footprint Capacitor_SMD:C_0805_2012Metric_Pad1.15x1.40mm_HandSolder -> Capacitor_SMD:C_0805_2012Metric
- C18: renamed from C24; footprint Capacitor_SMD:C_0805_2012Metric_Pad1.18x1.45mm_HandSolder -> Capacitor_SMD:C_0805_2012Metric
- C19: renamed from C6; footprint Capacitor_SMD:C_0805_2012Metric_Pad1.15x1.40mm_HandSolder -> Capacitor_SMD:C_0805_2012Metric
- C20: renamed from C7; footprint Capacitor_SMD:C_0805_2012Metric_Pad1.15x1.40mm_HandSolder -> Capacitor_SMD:C_0805_2012Metric
- C21: renamed from C16; footprint Capacitor_SMD:C_0805_2012Metric_Pad1.18x1.45mm_HandSolder -> Capacitor_SMD:C_0805_2012Metric
- C23: renamed from C20; footprint Capacitor_SMD:C_0805_2012Metric_Pad1.18x1.45mm_HandSolder -> Capacitor_SMD:C_0805_2012Metric
- C24: renamed from C21; footprint Capacitor_SMD:C_0805_2012Metric_Pad1.18x1.45mm_HandSolder -> Capacitor_SMD:C_0805_2012Metric
- F1: renamed from F3; JLC Part# C883109 -> (none)
- J7, J8: footprint Connector_PinHeader_2.54mm:PinHeader_1x02_P2.54mm_Vertical -> Jumper:SolderJumper-2_P1.3mm_Open_RoundedPad1.0x1.5mm
- renumbered C23 to C22, D1 to D3, D2 to D4, J3 to J10, J9 to J11
Connections:
- net +5V: now also J3.25 (P25)
- net ACK: now also J3.5
- net ATN: now also J3.17 (P17)
- net BSY: now also J3.6
- net CD: now also J3.15 (P15)
- net DB0: now also J3.8
- net DB1: now also J3.21 (P21)
- net DB2: now also J3.22 (P22)
- net DB3: now also J3.10
- net DB4: now also J3.23 (P23)
- net DB5: now also J3.11
- net DB6: now also J3.12
- net DB7: now also J3.13
- net DBP: now also J3.20 (P20)
- net GND: now also J3.0 (PAD), J3.14 (P14), J3.16 (P16), J3.18 (P18), J3.24 (P24), J3.7, J3.9
- net IO: now also J3.3
- net MSG: now also J3.2
- net REQ: now also J3.1
- net RST: now also J3.4
- net SEL: now also J3.19 (P19)

Commit message: intermediate - horizonal r's
Connections:
- no-connect marks 0 -> 1
Other:
- moved on the sheet: C21, C22, D4, F2, J10, J8

Commit message: initial rough parts placement
Parts:
- removed J11: Conn_01x02_Male, Connector_PinHeader_2.54mm:PinHeader_1x02_P2.54mm_Vertical, symbol Connector:Conn_01x02_Male
Other:
- note removed: "Mysterious Connector"
Changed lines of the file:
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@@
 	)
 	(junction
-		(at 85.725 144.145)
-		(diameter 0)
-		(color 0 0 0 0)
-	)
-	(junction
 		(at 229.235 64.77)
 		(diameter 0)
@@
 	(wire
 		(pts
-			(xy 85.725 146.685) (xy 85.725 144.145)
-		)
-		(stroke
-			(width 0)
-			(type default)
-		)
-	)
-	(wire
-		(pts
 			(xy 114.3 76.2) (xy 121.285 76.2)
 		)
@@
 	(wire
 		(pts
-			(xy 85.725 144.145) (xy 90.805 144.145)
-		)
-		(stroke
-			(width 0)
-			(type default)
-		)
-	)
-	(wire
-		(pts
 			(xy 86.36 88.265) (xy 86.36 92.075)
 		)
@@
 	(polyline
 		(pts
-			(xy 68.58 157.48) (xy 101.6 157.48)
-		)
-		(stroke
-			(width 0)
-			(type default)
-		)
-	)
-	(polyline
-		(pts
 			(xy 276.86 85.725) (xy 206.375 85.725)
 		)
@@
 		)
 	)
-	(polyline
-		(pts
-			(xy 101.6 157.48) (xy 101.6 133.985)
-		)
-		(stroke
-			(width 0)
-			(type default)
-		)
-	)
 	(wire
 		(pts
@@
 		)
 	)
-	(wire
-		(pts
-			(xy 90.805 144.145) (xy 90.805 145.415)
-		)
-		(stroke
-			(width 0)
-			(type default)
-		)
-	)
 	(polyline
 		(pts
@@
 		)
 	)
-	(polyline
-		(pts
-			(xy 68.58 133.985) (xy 68.58 157.48)
-		)
-		(stroke
-			(width 0)
-			(type default)
-		)
-	)
-	(polyline
-		(pts
-			(xy 68.58 133.985) (xy 101.6 133.985)
-		)
-		(stroke
-			(width 0)
-			(type default)
-		)
-	)
 	(wire
 		(pts
@@
 		)
 	)
-	(text "Mysterious Connector"
-		(exclude_from_sim no)
-		(at 74.295 154.94 0)
-		(effects
-			(font
-				(size 1.27 1.27)
-			)
-			(justify left bottom)
-		)
-	)
 	(text "More Decoupling Caps"
 		(exclude_from_sim no)
@@
 	)
 	(symbol
-		(lib_id "power:GND")
-		(at 90.805 145.415 0)
-		(unit 1)
-		(exclude_from_sim no)
-		(in_bom yes)
-		(on_board yes)
-		(dnp no)
-		(property "Reference" "#PWR085"
-			(at 90.805 151.765 0)
-			(effects
-				(font
-					(size 1.27 1.27)
-				)
-				(hide yes)
-			)
-		)
-		(property "Value" "GND"
-			(at 90.932 149.8092 0)
-			(effects
-				(font
-					(size 1.27 1.27)
-				)
-			)
-		)
-		(property "Footprint" ""
-			(at 90.805 145.415 0)
-			(effects
-				(font
-					(size 1.27 1.27)
-				)
-				(hide yes)
-			)
-		)
-		(property "Datasheet" ""
-			(at 90.805 145.415 0)
-			(effects
-				(font
-					(size 1.27 1.27)
-				)
-				(hide yes)
-			)
-		)
-		(property "Description" ""
-			(at 90.805 145.415 0)
-			(effects
-				(font
-					(size 1.27 1.27)
-				)
-				(hide yes)
-			)
-		)
-		(pin "1"
-		)
-		(instances
-			(project "Desktop_50_Pin_TopConn"
-				(path "/e40e8cef-4fb0-4fc3-be09-3875b2cc8469/f03a5fc0-9798-4033-842c-4371c8fa3a63"
-					(reference "#PWR085")
-					(unit 1)
-				)
-			)
-		)
-	)
-	(symbol
 		(lib_id "Device:CP")
 		(at 76.2 71.755 0)
@@
 					(unit 1)
 				)
-			)
-		)
-	)
-	(symbol
-		(lib_id "Connector:Conn_01x02_Male")
-		(at 80.645 144.145 0)
-		(unit 1)
-		(exclude_from_sim no)
-		(in_bom yes)
-		(on_board yes)
-		(dnp no)
-		(property "Reference" "J11"
-			(at 78.105 145.415 0)
-			(effects
-				(font
-					(size 1.27 1.27)
-				)
-			)
-		)
-		(property "Value" "Conn_01x02_Male"
-			(at 80.645 149.225 0)
-			(effects
-				(font
-					(size 1.27 1.27)
-				)
-			)
-		)
-		(property "Footprint" "Connector_PinHeader_2.54mm:PinHeader_1x02_P2.54mm_Vertical"
-			(at 80.645 144.145 0)
-			(effects
-				(font
-					(size 1.27 1.27)
-				)
-				(hide yes)
-			)
-		)
-		(property "Datasheet" "~"
-			(at 80.645 144.145 0)
-			(effects
-				(font
-					(size 1.27 1.27)
-				)
-				(hide yes)
-			)
-		)
-		(property "Description" ""
-			(at 80.645 144.145 0)
-			(effects
-				(font
-					(size 1.27 1.27)
-				)
-				(hide yes)
-			)
-		)
-		(pin "1"
-		)
-		(pin "2"
-		)
-		(instances
-			(project "Desktop_50_Pin_TopConn"
-				(path "/e40e8cef-4fb0-4fc3-be09-3875b2cc8469/f03a5fc0-9798-4033-842c-4371c8fa3a63"
-					(reference "J11")
-					(unit 1)
-				)

Commit message: more routing
Parts:
- C13, C14, C15, C16, C18, C23: footprint Capacitor_SMD:C_0805_2012Metric -> Capacitor_SMD:C_0402_1005Metric; LCSC (none) -> C307331
- C17, C19, C20, C21, C24: footprint Capacitor_SMD:C_0805_2012Metric -> Capacitor_SMD:C_0603_1608Metric; LCSC (none) -> C1705
- C22: footprint Capacitor_SMD:C_1206_3216Metric -> Capacitor_SMD:C_0603_1608Metric; LCSC (none) -> C59461
- D3, D4: value D -> Schottky Diode; footprint Diode_SMD:D_SMA -> Diode_SMD:D_SOD-123; LCSC (none) -> C8598
- F1, F2: LCSC (none) -> C883111
- J10, J7, J8: LCSC (none) -> --
- J3: footprint Connector_Dsub:DSUB-25_Male_Horizontal_P2.77x2.84mm_EdgePinOffset4.94mm_Housed_MountingHolesOffset7.48mm -> Connector_Dsub:DSUB-25_Male_EdgeMount_P2.77mm; symbol Connector:DB25_Plug_MountingHoles -> Connector:DB25_Plug; LCSC (none) -> C75745
Connections:
- net GND: no longer J3.0 (PAD)

Commit message: as-ordered PROTOTYPE
Parts:
- removed C19: 4.7uF, Capacitor_SMD:C_0603_1608Metric, symbol Device:CP
- removed C20, C21, C24: 4.7uF, Capacitor_SMD:C_0603_1608Metric, symbol Device:C
- removed C22: 20uF, Capacitor_SMD:C_0603_1608Metric, symbol Device:CP
- removed C23: 0.1uF, Capacitor_SMD:C_0402_1005Metric, symbol Device:C
- removed F2: Polyfuse, Fuse:Fuse_0805_2012Metric_Pad1.15x1.40mm_HandSolder, symbol Device:Polyfuse
- removed J7: TERM_BCKF, Jumper:SolderJumper-2_P1.3mm_Open_RoundedPad1.0x1.5mm, symbol Connector:Conn_01x02_Male
- removed J8: EPWR, Jumper:SolderJumper-2_P1.3mm_Open_RoundedPad1.0x1.5mm, symbol Connector:Conn_01x02_Male
- added C10, C23, C43: 0.1uF, Capacitor_SMD:C_0402_1005Metric, symbol Device:C_Small
- added C19, C20, C24, C25, C26, C9: 25V 10uF, Capacitor_SMD:C_0603_1608Metric, symbol Device:C_Small
- added C22, C8: 4.7uF, Capacitor_SMD:C_0603_1608Metric, symbol Device:C_Small
- added D8, D9: Schottky Diode, Diode_SMD:D_SOD-123, symbol Device:D
- added F3, F4, F5: Polyfuse, Fuse:Fuse_0805_2012Metric_Pad1.15x1.40mm_HandSolder, symbol Device:Polyfuse
- added JP3: USB Pwr En, Jumper:SolderJumper-2_P1.3mm_Open_TrianglePad1.0x1.5mm, symbol Jumper:SolderJumper_2_Open
- added JP4: Berg Pwr En, Jumper:SolderJumper-2_P1.3mm_Open_TrianglePad1.0x1.5mm, symbol Jumper:SolderJumper_2_Open
- added JP5: Term Input Pwr En, Jumper:SolderJumper-2_P1.3mm_Open_TrianglePad1.0x1.5mm, symbol Jumper:SolderJumper_2_Open
- added JP6: Term Output En, Jumper:SolderJumper-2_P1.3mm_Open_TrianglePad1.0x1.5mm, symbol Jumper:SolderJumper_2_Open
- added U10: AMS1117-2.85, Package_TO_SOT_SMD:SOT-223-3_TabPin2, symbol Regulator_Linear:AMS1117CD-2.85
- added U11: AMS1117-3.3, Package_TO_SOT_SMD:SOT-223-3_TabPin2, symbol Regulator_Linear:AMS1117-3.3
- C13, C14, C15, C16, C18: symbol Device:C -> Device:C_Small
- D4: value Schottky Diode -> Schottky
- J3: value DB25_Plug_MountingHoles -> SCSI Connector
Connections:
- net +2V8: now also C10.1, C24.1, C9.1, U10.2 (VO)
- net +3V3: now also C25.1, C26.1, C43.1, U11.2 (VO)
- net +5V: now also C19.1, C20.1, C22.1, C23.2, C8.1, JP3.2 (B), JP4.2 (B), JP5.2 (B), JP6.1 (A), U10.3 (VI), U11.3 (VI); no longer D3.2 (A), J3.25 (P25)
- net GND: now also C10.2, C19.2, C20.2, C22.2, C23.1, C24.2, C25.2, C26.2, C43.2, C8.2, C9.2, U10.1 (GND), U11.1 (GND)
- net at J10.1 (5V): now also F4.2; no longer D4.2 (A)
- net at F1.2: now also D3.1 (K)
- new net: D8.2 (A), F3.1
- new net: D8.1 (K), JP3.1 (A)
- new net: D9.1 (K), JP5.1 (A)
- new net: D9.2 (A), F5.1
- new net: D4.2 (A), F4.1
- new net: D4.1 (K), JP4.1 (A)
- new net: D3.2 (A), JP6.2 (B)
- new net EXT_TERM_PWR: F1.1, F5.2, J3.25 (P25)
- new net VBUS: F3.2
Other:
- note added: "Depending upon the use case, EXT TERM PWR could be an input or an output"
- note added: "Digital Logic Voltage"
- note added: "Enable ONE power input"
- note added: "Termination Voltage"
- note added: "USB Power Input"
- note removed: "Decoupling Caps"
- note removed: "Power Distribution Network"
- moved on the sheet: C13, C14, C15, C16, C17, C18, D4, J10, J3
