File: hardware/USB_Bridge/piccolo.kicad_sch (KiCad schematic)
At the start: 44 parts, among them J1 USB_C_Receptacle_USB2.0, J2 CON_PICO_40W, J3 Debug, Q1 DMG1012T, SW2 TS-1187A-B-A-B, U1 W25Q16JVUXIQ, U3 RP2040, U4 AMS1117-3.3, X1 SIT1602AI-22-33E-12.000000, Y1 12MHz

Commit message: intermediate checkin
Parts:
- removed J2: CON_PICO_40W, agausmann:RaspberryPi_Pico_OutlineAndPads, symbol Connector_Generic:Conn_02x20_Counter_Clockwise
- added JP10, JP11, JP12, JP13, JP14, JP15, JP16, JP17, JP18, JP19, JP20, JP21, JP22, JP23, JP24, JP25, JP26, JP27, JP28, JP29, JP3, JP30, JP31, JP32, JP33, JP34, JP35, JP36, JP37, JP38, JP39, JP4, JP40, JP41, JP42, JP43, JP44, JP45, JP46, JP5, JP6, JP7, JP8, JP9: SolderJumper_2_Bridged, Jumper:SolderJumper-2_P1.3mm_Bridged_RoundedPad1.0x1.5mm, symbol Jumper:SolderJumper_2_Bridged
- C1, C10, C11, C12, C13, C14, C15, C16, C17, C2, C4, C5, C6, C7, C8, C9: Manufacturer Samsung -> (none)
- C3: Manufacturer Kyocera -> (none)
- D1: Manufacturer onsemi -> (none)
- D2, D3: Manufacturer Lite-On -> (none)
- J1: Manufacturer Korean Hroparts -> (none)
- Q1: Manufacturer Diodes Inc -> (none)
- R10, R11, R13, R14, R15, R2, R3, R4, R5, R6, R7, R8: Manufacturer Yageo -> (none)
- R12: Manufacturer Stackpole -> (none)
- SW2: MANUFACTURER XKB Industrial Precision -> (none); MAXIMUM_PACKAGE_HEIGHT 1.5mm -> (none); PARTREV A0 -> (none); STANDARD Manufacturer Recommendations -> (none)
- U1: Manufacturer Winbond -> (none)
- U3: Manufacturer Raspberry Pi -> (none)
- X1: Manufacturer SiTime -> (none)
Connections:
- net GND: now also JP45.1 (A); no longer U3.19 (TESTEN)
- net GPIO0: now also JP4.2 (B); no longer U3.2 (GPIO0)
- net GPIO1: now also JP6.2 (B); no longer U3.3 (GPIO1)
- net GPIO10: now also JP23.2 (B); no longer U3.13 (GPIO10)
- net GPIO11: now also JP24.2 (B); no longer U3.14 (GPIO11)
- net GPIO12: now also JP26.2 (B); no longer U3.15 (GPIO12)
- net GPIO13: now also JP28.2 (B); no longer U3.16 (GPIO13)
- net GPIO14: now also JP30.2 (B); no longer U3.17 (GPIO14)
- net GPIO15: now also JP32.2 (B); no longer U3.18 (GPIO15)
- net GPIO16: now also JP35.2 (B); no longer U3.27 (GPIO16)
- net GPIO17: now also JP36.2 (B); no longer U3.28 (GPIO17)
- net GPIO18: now also JP38.2 (B); no longer U3.29 (GPIO18)
- net GPIO19: now also JP40.2 (B); no longer U3.30 (GPIO19)
- net GPIO2: now also JP8.2 (B); no longer U3.4 (GPIO2)
- net GPIO20: now also JP41.2 (B); no longer U3.31 (GPIO20)
- net GPIO21: now also JP43.2 (B); no longer U3.32 (GPIO21)
- net GPIO22: now also JP44.2 (B); no longer U3.34 (GPIO22)
- net GPIO23: now also JP46.2 (B); no longer U3.35 (GPIO23)
- net GPIO24: now also JP3.1 (A); no longer U3.36 (GPIO24)
- net GPIO25: now also JP5.1 (A); no longer U3.37 (GPIO25)
- net GPIO26_ADC0: now also JP7.1 (A); no longer U3.38 (GPIO26/ADC0)
- net GPIO27_ADC1: now also JP9.1 (A); no longer U3.39 (GPIO27/ADC1)
- net GPIO28_ADC2: now also JP11.1 (A); no longer U3.40 (GPIO28/ADC2)
- net GPIO29_ADC3: now also JP13.1 (A); no longer U3.41 (GPIO29/ADC3)
- net GPIO3: now also JP10.2 (B); no longer U3.5 (GPIO3)
- net GPIO4: now also JP12.2 (B); no longer U3.6 (GPIO4)
- net GPIO5: now also JP14.2 (B); no longer U3.7 (GPIO5)
- net GPIO6: now also JP15.2 (B); no longer U3.8 (GPIO6)
- net GPIO7: now also JP17.2 (B); no longer U3.9 (GPIO7)
- net GPIO8: now also JP19.2 (B); no longer U3.11 (GPIO8)
- net GPIO9: now also JP21.2 (B); no longer U3.12 (GPIO9)
- net QSPI_SCLK: now also JP33.1 (A); no longer U3.52 (QSPI_SCLK)
- net QSPI_SD0: now also JP25.1 (A); no longer U3.53 (QSPI_SD0)
- net QSPI_SD1: now also JP27.1 (A); no longer U3.55 (QSPI_SD1)
- net QSPI_SD2: now also JP29.1 (A); no longer U3.54 (QSPI_SD2)
- net QSPI_SD3: now also JP31.1 (A); no longer U3.51 (QSPI_SD3)
- net QSPI_SS: now also JP34.1 (A); no longer U3.56 (QSPI_SS_N)
- net RUN: now also JP42.1 (A); no longer U3.26 (RUN)
- net SWCLK: now also JP37.1 (A); no longer U3.24 (SWCLK)
- net SWDIO: now also JP39.1 (A); no longer U3.25 (SWDIO)
- net XIN: now also JP20.1 (A); no longer U3.20 (XIN)
- net XOUT: now also JP22.1 (A); no longer U3.21 (XOUT)
- net at R11.2: now also JP16.1 (A); no longer U3.46 (USB_DM)
- net at R10.2: now also JP18.1 (A); no longer U3.47 (USB_DP)
- new net: JP34.2 (B), U3.56 (QSPI_SS_N)
- new net: JP17.1 (A), U3.9 (GPIO7)
- new net: JP13.2 (B), U3.41 (GPIO29/ADC3)
- new net: JP12.1 (A), U3.6 (GPIO4)
- new net: JP31.2 (B), U3.51 (QSPI_SD3)
- new net: JP22.2 (B), U3.21 (XOUT)
- new net: JP8.1 (A), U3.4 (GPIO2)
- new net: JP38.1 (A), U3.29 (GPIO18)
- new net: JP10.1 (A), U3.5 (GPIO3)
- new net: JP37.2 (B), U3.24 (SWCLK)
- new net: JP41.1 (A), U3.31 (GPIO20)
- new net: JP7.2 (B), U3.38 (GPIO26/ADC0)
- new net: JP19.1 (A), U3.11 (GPIO8)
- new net: JP11.2 (B), U3.40 (GPIO28/ADC2)
- new net: JP18.2 (B), U3.47 (USB_DP)
- new net: JP20.2 (B), U3.20 (XIN)
- new net: JP27.2 (B), U3.55 (QSPI_SD1)
- new net: JP39.2 (B), U3.25 (SWDIO)
- new net: JP25.2 (B), U3.53 (QSPI_SD0)
- new net: JP44.1 (A), U3.34 (GPIO22)
- new net: JP6.1 (A), U3.3 (GPIO1)
- new net: JP21.1 (A), U3.12 (GPIO9)
- new net: JP3.2 (B), U3.36 (GPIO24)
- new net: JP29.2 (B), U3.54 (QSPI_SD2)
- new net: JP14.1 (A), U3.7 (GPIO5)
- new net: JP23.1 (A), U3.13 (GPIO10)
- new net: JP45.2 (B), U3.19 (TESTEN)
- new net: JP32.1 (A), U3.18 (GPIO15)
- new net: JP30.1 (A), U3.17 (GPIO14)
- new net: JP43.1 (A), U3.32 (GPIO21)
- new net: JP35.1 (A), U3.27 (GPIO16)
- new net: JP5.2 (B), U3.37 (GPIO25)
- new net: JP26.1 (A), U3.15 (GPIO12)
- new net: JP16.2 (B), U3.46 (USB_DM)
- new net: JP46.1 (A), U3.35 (GPIO23)
- new net: JP24.1 (A), U3.14 (GPIO11)
- new net: JP28.1 (A), U3.16 (GPIO13)
- new net: JP4.1 (A), U3.2 (GPIO0)
- new net: JP42.2 (B), U3.26 (RUN)
- new net: JP36.1 (A), U3.28 (GPIO17)
- new net: JP40.1 (A), U3.30 (GPIO19)
- new net: JP9.2 (B), U3.39 (GPIO27/ADC1)
- new net: JP33.2 (B), U3.52 (QSPI_SCLK)
- new net: JP15.1 (A), U3.8 (GPIO6)

Commit message: intermediate - horizonal r's
Parts:
- added J13: Conn_01x03_Male, Jumper:SolderJumper-3_P1.3mm_Open_RoundedPad1.0x1.5mm, symbol Connector:Conn_01x03_Male
- added R79, R80, R81, R82, R83, R84, R85, R86, R87, R88, R89, R90, R91, R92, R93, R94, R95, R96: 1k, Resistor_SMD:R_0402_1005Metric, symbol Device:R
- added TP1: TestPoint_Small, TestPoint:TestPoint_Pad_D1.0mm, symbol Connector:TestPoint_Small
Connections:
- net RUN: now also TP1.1
- net GPIO0 renamed GPIO00
- net GPIO00: now also R96.1
- net GPIO1 renamed GPIO01
- net GPIO01: now also R95.1
- net GPIO10 renamed SD_CLK
- net GPIO11 renamed SD_CMD_MOSI
- net GPIO12 renamed SD_D0_MISO
- net GPIO13 renamed SD_D1
- net GPIO14 renamed SD_D2
- net GPIO15 renamed SD_D3_CS
- net GPIO16 renamed SDA
- net GPIO17 renamed SCL
- net GPIO18 renamed oCD_iSEL
- net oCD_iSEL: now also J13.2 (Pin_2)
- net GPIO19 renamed oREQ
- net oREQ: now also R81.1
- net GPIO2 renamed GPIO02
- net GPIO02: now also R93.1
- net GPIO20 renamed oMSG_iBSY
- net oMSG_iBSY: now also R82.2
- net GPIO21 renamed oSEL
- net oSEL: now also R83.2
- net GPIO22 renamed oIO
- net oIO: now also R84.2
- net GPIO26_ADC0 renamed oACK
- net oACK: now also R86.1
- net GPIO27_ADC1 renamed oBSY
- net GPIO28_ADC2 renamed GPIO28
- net GPIO28: now also R90.1, R94.1
- net GPIO3 renamed GPIO03
- net GPIO03: now also R92.1
- net GPIO4 renamed GPIO04
- net GPIO04: now also R91.1
- net GPIO5 renamed GPIO05
- net GPIO05: now also R89.1
- net GPIO6 renamed GPIO06
- net GPIO06: now also R88.1
- net GPIO7 renamed GPIO07
- net GPIO07: now also R87.1
- net GPIO8 renamed GPIO08
- net GPIO08: now also R85.1
- net GPIO9 renamed DBPTr
- new net: J13.1 (Pin_1), R80.2
- new net: J13.3 (Pin_3), R79.2
- new net DB0T: R96.2
- new net DB1T: R95.2
- new net DB2T: R93.2
- new net DB3T: R92.2
- new net DB4T: R91.2
- new net DB5T: R89.2
- new net DB6T: R88.2
- new net DB7T: R87.2
- new net DBPT: R85.2
- new net iACK: R86.2
- new net iATN: R90.2
- new net iBSY: R82.1
- new net iCD: R80.1
- new net iIO: R84.1
- new net iMSG: R94.2
- new net iREQ: R81.2
- new net iRST: R83.1
- new net iSEL: R79.1
Other:
- note added: "NEED DIFFERENT FLASH DEVICE!!!!!!!!!"
- note added: "Series current-limiter Necessary for LVT and LVTH"
- moved on the sheet: C17, C3, D2, D3, J3, Q1, R14, R15, R7, R8, X1

Commit message: initial rough parts placement
Parts:
- removed C17: 100n 6.3V, Capacitor_SMD:C_0402_1005Metric, symbol Device:C_Small
- removed JP10, JP11, JP12, JP13, JP14, JP15, JP16, JP17, JP18, JP19, JP20, JP21, JP22, JP23, JP24, JP25, JP26, JP27, JP28, JP29, JP3, JP30, JP31, JP32, JP33, JP34, JP35, JP36, JP37, JP38, JP39, JP4, JP40, JP41, JP42, JP43, JP44, JP45, JP46, JP5, JP6, JP7, JP8, JP9: SolderJumper_2_Bridged, Jumper:SolderJumper-2_P1.3mm_Bridged_RoundedPad1.0x1.5mm, symbol Jumper:SolderJumper_2_Bridged
- removed X1: SIT1602AI-22-33E-12.000000, Crystal:Crystal_SMD_SeikoEpson_TSX3225-4Pin_3.2x2.5mm, symbol agausmann:SIT1602
- added R1: 1k, Resistor_SMD:R_0402_1005Metric, symbol Device:R
- added SW3: SW_MEC_5E, Library:TS-1187A-B-A-B, symbol Switch:SW_MEC_5E
- R12: footprint Resistor_SMD:R_0603_1608Metric -> Resistor_SMD:R_0402_1005Metric
Connections:
- net +3V3: now also R1.1
- net DBPTr: now also U3.12 (GPIO9)
- net GND: now also U3.19 (TESTEN), SW3.1 (2)
- net GPIO00: now also U3.2 (GPIO0)
- net GPIO01: now also U3.3 (GPIO1)
- net GPIO02: now also U3.4 (GPIO2)
- net GPIO03: now also U3.5 (GPIO3)
- net GPIO04: now also U3.6 (GPIO4)
- net GPIO05: now also U3.7 (GPIO5)
- net GPIO06: now also U3.8 (GPIO6)
- net GPIO07: now also U3.9 (GPIO7)
- net GPIO08: now also U3.11 (GPIO8)
- net GPIO23: now also U3.35 (GPIO23)
- net GPIO24: now also U3.36 (GPIO24)
- net GPIO25: now also U3.37 (GPIO25)
- net GPIO28: now also U3.40 (GPIO28/ADC2)
- net GPIO29_ADC3: now also U3.41 (GPIO29/ADC3)
- net QSPI_SCLK: now also U3.52 (QSPI_SCLK)
- net QSPI_SD0: now also U3.53 (QSPI_SD0)
- net QSPI_SD1: now also U3.55 (QSPI_SD1)
- net QSPI_SD2: now also U3.54 (QSPI_SD2)
- net QSPI_SD3: now also U3.51 (QSPI_SD3)
- net QSPI_SS: now also U3.56 (QSPI_SS_N)
- net RUN: now also U3.26 (RUN), R1.2, SW3.2 (K)
- net SCL: now also U3.28 (GPIO17)
- net SDA: now also U3.27 (GPIO16)
- net SD_CLK: now also U3.13 (GPIO10)
- net SD_CMD_MOSI: now also U3.14 (GPIO11)
- net SD_D0_MISO: now also U3.15 (GPIO12)
- net SD_D1: now also U3.16 (GPIO13)
- net SD_D2: now also U3.17 (GPIO14)
- net SD_D3_CS: now also U3.18 (GPIO15)
- net SWCLK: now also U3.24 (SWCLK)
- net SWDIO: now also U3.25 (SWDIO)
- net XIN: now also U3.20 (XIN)
- net XOUT: now also U3.21 (XOUT)
- net oACK: now also U3.38 (GPIO26/ADC0)
- net oBSY: now also U3.39 (GPIO27/ADC1)
- net oCD_iSEL: now also U3.29 (GPIO18)
- net oIO: now also U3.34 (GPIO22)
- net oMSG_iBSY: now also U3.31 (GPIO20)
- net oREQ: now also U3.30 (GPIO19)
- net oSEL: now also U3.32 (GPIO21)
- net at R11.2: now also U3.46 (USB_DM)
- net at R10.2: now also U3.47 (USB_DP)
Other:
- note added: "MCU Reset"
- note removed: "Prefer MEMS oscillators over crystals"

Commit message: more routing
Parts:
- added C40, C42: 15p, Capacitor_SMD:C_0603_1608Metric, symbol Device:C_Small
- added R2: 1k, Resistor_SMD:R_0402_1005Metric, symbol Device:R
- added SD1: Micro SD Card, Connector_Card:microSD_HC_Molex_104031-0811, symbol Connector:Micro_SD_Card_Det2
- C10, C11, C13, C15, C2, C5, C7, C8, C9: value 100n 6.3V -> 0.1uF; LCSC C1525 -> C307331
- C4, C6: footprint Capacitor_SMD:C_0805_2012Metric -> Capacitor_SMD:C_0402_1005Metric; LCSC C440198 -> C15525
- D1: value MBR120VLSFT1G -> Schottky Diode; footprint Diode_SMD:D_SOD-123F -> Diode_SMD:D_SOD-123; LCSC C123070 -> C8598
- D2: footprint LED_SMD:LED_0603_1608Metric -> LED_SMD:LED_0805_2012Metric; LCSC C72043 -> C2297
- D3: footprint LED_SMD:LED_0603_1608Metric -> LED_SMD:LED_0805_2012Metric; LCSC C72043 -> C84256
- J1: footprint Connector_USB:USB_C_Receptacle_HRO_TYPE-C-31-M-12 -> Connector_USB:USB_C_Receptacle_G-Switch_GT-USB-7010ASV
- J13, J3, R1, TP1: LCSC (none) -> --
- R1, R79, R80, R81, R82, R83, R84, R85, R86, R87, R88, R89, R90, R91, R92, R93, R94, R95, R96: LCSC (none) -> C11702
- R10, R11: footprint Resistor_SMD:R_0201_0603Metric -> Resistor_SMD:R_0402_1005Metric
- SW2: value TS-1187A-B-A-B -> USB Boot; footprint SW_TS-1187A-B-A-B -> Button_Switch_SMD:SW_Push_1P1T_XKB_TS-1187A; symbol TS-1187A-B-A-B:TS-1187A-B-A-B -> Switch:SW_Push; LCSC (none) -> C318884
- SW3: value SW_MEC_5E -> RP2040 Reset; footprint Library:TS-1187A-B-A-B -> Button_Switch_SMD:SW_Push_1P1T_XKB_TS-1187A; symbol Switch:SW_MEC_5E -> Switch:SW_Push; LCSC (none) -> C318884
- U1: footprint agausmann:USON-8-1EP_3x2mm_P0.5mm_EP0.2x1.6mm -> Package_SON:Winbond_USON-8-1EP_3x2mm_P0.5mm_EP0.2x1.6mm; LCSC C152595 -> C2843335
- Y1: LCSC (none) -> C20625731
Connections:
- net +3V3: now also SD1.4 (VDD)
- net GND: now also SW2.1, C40.2, C42.2, SD1.11 (SHIELD), SD1.6 (VSS); no longer SW2.A, SW2.B
- net SD_CLK: now also SD1.5 (CLK)
- net SD_CMD_MOSI: now also SD1.3 (CMD)
- net SD_D0_MISO: now also SD1.7 (DAT0)
- net SD_D1: now also SD1.8 (DAT1)
- net SD_D2: now also SD1.1 (DAT2)
- net SD_D3_CS: now also SD1.2 (DAT3/CD)
- net XIN: now also C42.1
- net XOUT: now also R2.1; no longer Y1.3
- new net: C40.1, R2.2, Y1.3
- new net: R2.2, SW2.2
- no-connect marks 3 -> 5
Other:
- note removed: "NEED DIFFERENT FLASH DEVICE!!!!!!!!!"
- note removed: "NOTE - Max clock rate is 80MHz System clock may have to be reduced to stay within spec for this chip."

Commit message: more routing fun....
Parts:
- removed TP1: TestPoint_Small, TestPoint:TestPoint_Pad_D1.0mm, symbol Connector:TestPoint_Small
- J3: footprint Connector_PinHeader_2.54mm:PinHeader_1x03_P2.54mm_Vertical -> Connector_PinHeader_2.54mm:PinHeader_1x03_P2.54mm_Vertical_SMD_Pin1Left
Changed lines of the file:
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@@
-	)
-	(symbol
-		(lib_id "Connector:TestPoint_Small")
-		(at 328.93 232.41 0)
-		(unit 1)
-		(exclude_from_sim no)
-		(in_bom yes)
-		(on_board yes)
-		(dnp no)
-		(property "Reference" "TP1"
-			(at 324.866 232.41 0)
-			(effects
-				(font
-					(size 1.27 1.27)
-				)
-				(justify left)
-			)
-		)
-		(property "Value" "TestPoint_Small"
-			(at 330.2 233.6799 0)
-			(effects
-				(font
-					(size 1.27 1.27)
-				)
-				(justify left)
-				(hide yes)
-			)
-		)
-		(property "Footprint" "TestPoint:TestPoint_Pad_D1.0mm"
-			(at 334.01 232.41 0)
-			(effects
-				(font
-					(size 1.27 1.27)
-				)
-				(hide yes)
-			)
-		)
-		(property "Datasheet" "~"
-			(at 334.01 232.41 0)
-			(effects
-				(font
-					(size 1.27 1.27)
-				)
-				(hide yes)
-			)
-		)
-		(property "Description" "test point"
-			(at 328.93 232.41 0)
-			(effects
-				(font
-					(size 1.27 1.27)
-				)
-				(hide yes)
-			)
-		)
-		(property "LCSC" "--"
-			(at 328.93 232.41 0)
-			(effects
-				(font
-					(size 1.27 1.27)
-				)
-				(hide yes)
-			)
-		)
-		(pin "1"
-		)
-		(instances
-			(project "Desktop_50_Pin_TopConn"
-				(path "/e40e8cef-4fb0-4fc3-be09-3875b2cc8469/e7b9a285-64df-429b-bf4b-655561da859b"
-					(reference "TP1")
-					(unit 1)
-				)
-			)
-		)
 	)
 	(symbol
@@
 			)
 		)
-		(property "Footprint" "Connector_PinHeader_2.54mm:PinHeader_1x03_P2.54mm_Vertical"
+		(property "Footprint" "Connector_PinHeader_2.54mm:PinHeader_1x03_P2.54mm_Vertical_SMD_Pin1Left"
 			(at 314.96 48.26 0)
 			(effects

Commit message: as-ordered PROTOTYPE
Parts:
- removed C3: 1n 25V, Capacitor_SMD:C_0402_1005Metric, symbol Device:C
- removed C4, C6: 10u 6.3V, Capacitor_SMD:C_0402_1005Metric, symbol Device:C_Small
- removed D1: Schottky Diode, Diode_SMD:D_SOD-123, symbol Device:D_Schottky
- removed Q1: DMG1012T, Package_TO_SOT_SMD:SOT-523, symbol Device:Q_NMOS_GSD
- removed R7: 200k, Resistor_SMD:R_0402_1005Metric, symbol Device:R
- removed R8: 100k, Resistor_SMD:R_0402_1005Metric, symbol Device:R
- removed U4: AMS1117-3.3, Package_TO_SOT_SMD:SOT-223-3_TabPin2, symbol Regulator_Linear:AMS1117-3.3
- added JP7: USB Bridge En, Jumper:SolderJumper-3_P1.3mm_Open_RoundedPad1.0x1.5mm, symbol Jumper:SolderJumper_3_Open
- added R3, R4: 1k, Resistor_SMD:R_0402_1005Metric, symbol Device:R
Connections:
- net +3V3: now also R3.1
- net GND: now also R4.2
- net GPIO29_ADC3: now also JP7.2 (C)
- new net: JP7.1 (A), R4.1
- new net: JP7.3 (B), R3.2
Other:
- note added: "Read mode from SD Card"
- note added: "USB Bridge Enable"
- note removed: "Replaced buck-boost with LDO regulator."
