File: hardware/USB_Bridge_v2/Usb_Bridge.kicad_pcb (KiCad board)
At the start: 4 copper layers, 50 x 36 mm, 147 parts, among them J1 ACK_En, J12 USB_C_Receptacle_USB2.0, J13 Conn_01x03_Male, J3 SCSI Connector, J4 SM04B-SRSS-TB(LF)(SN), J6 Conn_01x03_Male, Q1 AO3401A, Q2 AO3401A, SW1 SCSI Reset, SW2 USB Boot, SW3 RP2040 Reset, U1 LVT125, U10 AMS1117-2.85, U11 AMS1117-3.3, U12 W25Q16JVUXIQ, U13 RP2040, U2 LVT125, U3 LVT125, U4 LVT125, U5 74HC14, U6 LVT245, U7 LVT245, U8 LVT245, U9 LVT245, Y1 12MHz

Commit message: as-ordered v2 board
Parts:
- removed REF** (x2): OSHW-Logo2_7.3x6mm_SilkScreen, Symbol:OSHW-Logo2_7.3x6mm_SilkScreen
- moved J4 3.96 mm to (145.0, 109.6), turned to -90 degrees
- moved C38 0.13 mm to (148.9, 101.2)
- moved C39 0.13 mm to (148.9, 102.2)
- turned G*** to 180 degrees
Routing:
- net GND: track 259.2 -> 281.7 mm, vias 51 -> 55
- net SDA: track 35.8 -> 31.1 mm
- net SD_D3_CS: track 30.5 -> 31.9 mm
- net SCL: track 31.5 -> 30.2 mm, vias 2 -> 4
- net Net-(JP7-A): track 26.9 -> 26.2 mm
- net SD_CMD_MOSI: track 39.8 -> 40.5 mm
Other:
- board text added: "v2024.12.1a"
- board text removed: "v2024.12.1"
